File: fmc-host/fmc-host.sch (EAGLE design)
At the start: 321 parts, among them J1 SMA002, J10 ASP-134488-01, J2 SMA002, J3 SMA002, J4 SMA002, J5 SMA002, J6 ESHF-105-01-L-D-SM-K-TR, J7 12226-8250-00FR, J8 95278-101A16LF, J9 FMC_SINGLE_WIDTH_MODULE, Q1 SI1012R, Q2 SI1012R, U1 SN74LVC2G34DCKR, U10 DS90UB934-Q1, U11 DS90UB934-Q1, U12 DS91M040, U13 AD5766BCPZ-RL7, U14 MCP47FEB02A0-E/ST, U15 LM4132AMF-2.5/NOPBCT-ND, U16 AD7617BSTZ, U17 AD5142BCPZ10, U18 LTM4622A, U19 TPS62293DRV, U2 SN65LVDS9638DGN, U20 TPS7A49, U21 TPS7A49, U22 TPS7A30, U23 24AA64ST, U24 LTM8049_BGA, U3 FIN1032MTCX, U4 LTC2875_DFN, U5 ADCMP600, U6 ADCMP600, U7 DG1412E, U8 DG1412E, U9 DG1412E, X2 OE-LOGO_7X5, X3 OE-LOGO_7X5

Commit message: ONIX FMC Host revision 1.5
- Lots of minor fixes after extensive testing of 1.4
- VITA-57 compliance
- Remove debug points
- Standalone 1.8V regulator for deserializers
- Lots of other small fixes
Parts:
- removed D10, D11: APFA3011-AK13/F, jonnew:LED_3X_SMD-6
- removed D9: KDZ4.3B, jonnew:Z-DIODE_SOD123
- removed J10: ASP-134488-01, jonnew:FMC_HPC_400_PIN_MALE
- removed R82: 165k, jonnew:R_0402
- removed R83: 178k, jonnew:R_0402
- removed R84, R85: 10k, jonnew:R_0402
- removed R86, R87: 73.2k, jonnew:R_0402
- removed SJ1, SJ2: (no value), jonnew:SJ2_0201
- removed U18: LTM4622A, jonnew:LTM4622_BGA
- removed X3: OE-LOGO_7X5, jonnew:OE-LOGO_7X5
- C100, C104, C132, C99: value 47uF -> 0.1uF; device jonnew:C_1210 -> jonnew:C_0402
- C101, C109, C113, C116, C117, C62, C69, C95: value 0.1uF -> 10uF; device jonnew:C_0402 -> jonnew:C_0805
- C102, C133: value 0.1uF -> 47uF; device jonnew:C_0402 -> jonnew:C_1210
- C106, C34, C70, C80, C91, C92: value 0.1uF -> 10uF; device jonnew:C_0402 -> jonnew:C_1206
- C107, C110, C111, C115, C61: value 10uF -> 0.1uF; device jonnew:C_0805 -> jonnew:C_0402
- C108, C120: device jonnew:C_1206 -> jonnew:C_0805
- C11, C20, C24, C50, C51, C57, C58: value 0.1uF -> 10nF
- C118, C71, C79: device jonnew:C_0805 -> jonnew:C_1206
- C122, C123: value 10uF -> 10nF; device jonnew:C_0805 -> jonnew:C_0402
- C125, C126, C59: value 10nF -> 10uF; device jonnew:C_0402 -> jonnew:C_0805
- C128, C129: value 10uF -> 0.1uF, 500V; device jonnew:C_0805 -> jonnew:C_1210
- C13, C22, C52, C53, C60, C84: value 10nF -> 0.1uF
- C26: value 10nF -> 10uF; device jonnew:C_0402 -> jonnew:C_1206
- C28: value 10uF -> 4.7nF; device jonnew:C_1206 -> jonnew:C_0402
- C30: value 4.7nF -> 0.1uF
- C38: value 10uF -> 47nF; device jonnew:C_1206 -> jonnew:C_0402
- C39: value 0.1uF -> 47nF
- C40: value 47nF -> 1uF; device jonnew:C_0402 -> jonnew:C_0805
- C41: value 47nF -> 0.1uF
- C44, C68, C78, C90: value 1uF -> 0.1uF; device jonnew:C_0805 -> jonnew:C_0402
- C5: value 4.7nF -> 10uF; device jonnew:C_0402 -> jonnew:C_1206
- C64: value 10uF -> 1uF
- C7, C83, C93: value 10uF -> 0.1uF; device jonnew:C_1206 -> jonnew:C_0402
- C74, C75: value 10uF -> 1uF; device jonnew:C_1206 -> jonnew:C_0805
- C77: value 1uF -> 10uF
- C82: value 10uF -> 10nF; device jonnew:C_1206 -> jonnew:C_0402
- C88: value 0.1uF -> 1uF; device jonnew:C_0402 -> jonnew:C_0805
- C94: value 10uF -> 47uF; device jonnew:C_1206 -> jonnew:C_1210
- C96: value 47uF -> 10uF; device jonnew:C_1210 -> jonnew:C_0805
- C97, C98: value 10uF -> 47uF; device jonnew:C_0805 -> jonnew:C_1210
- D1, D2: value HSMG-C280 -> SESD0402X1UN-0020-090; device jonnew:LED_0402 -> jonnew:Z-DIODE_0402P-DFN
- D3: value HSMG-C280 -> BAR66; device jonnew:LED_0402 -> jonnew:DIODE2_SOT23
- D4, D5: value SESD0402X1UN-0020-090 -> BAR66; device jonnew:Z-DIODE_0402P-DFN -> jonnew:DIODE2_SOT23
- D6: value BAR66 -> KDZ4.3B; device jonnew:DIODE2_SOT23 -> jonnew:Z-DIODE_SOD123
- D7, D8: value BAR66 -> APFA3011-AK13/F; device jonnew:DIODE2_SOT23 -> jonnew:LED_3X_SMD-6
- J8: value 95278-101A16LF -> FMC_SINGLE_WIDTH_MODULE; device jonnew:PINHD-2X8_SMD -> jonnew:FMC_SINGLE_WIDTH_MODULE
- J9: value FMC_SINGLE_WIDTH_MODULE -> ASP-134488-01; device jonnew:FMC_SINGLE_WIDTH_MODULE -> jonnew:FMC_HPC_400_PIN_MALE
- L13: value (none) -> 1277AS-H-6R8M=P2
- R1: value 2k -> 3k
- R10, R9: value 150,0.25W -> 2k; device jonnew:R_0603 -> jonnew:R_0402
- R12, R6, R7: value 2k -> 150,0.25W; device jonnew:R_0402 -> jonnew:R_0603
- R13: value 2k -> 165k
- R14: value 150,0.25W -> 165k; device jonnew:R_0603 -> jonnew:R_0402
- R15: value 150,0.25W -> 10k; device jonnew:R_0603 -> jonnew:R_0402
- R16: value 165k -> 10k
- R17: value 165k -> 1k
- R18, R41: value 10k -> 1k
- R19: value 10k -> 5.6k 1%
- R2, R38, R39: value 4.7k -> 3k
- R20: value 1k -> 21k 1%
- R21: value 1k -> 5.6k 1%
- R22: value 5.6k 1% -> 21k 1%
- R23: value 21k 1% -> 49.9
- R24: value 5.6k 1% -> 49.9
- R25: value 21k 1% -> 100
- R26, R27: value 60 1% -> 100
- R3: value 4.7k -> 2k
- R30, R31, R32: value 100 -> 4.7k
- R33: value 3k -> 4.7k
- R34: value 49.9 -> DNP
- R35: value 49.9 -> 10k
- R36: value 4.7k -> DNP
- R37, R79: value 4.7k -> 10k
- R4: value 3k -> 2k
- R40: value DNP -> 4.7k
- R42: value DNP -> 1k
- R43, R71, R73: value 10k -> 4.7k
- R44, R45: value 3k -> 1k
- R46: value 4.7k -> 1k
- R48: value 1k -> 0
- R49: value 4.7k -> 165k
- R5: value 3k -> 150,0.25W; device jonnew:R_0402 -> jonnew:R_0603
- R50, R51, R52: value 1k -> 165k
- R53: value 1k -> 2.2k; device jonnew:R_0402 -> jonnew:RN2X8_1506
- R54: value 0 -> 2.2k; device jonnew:R_0402 -> jonnew:RN2X8_1506
- R55, R56: value 165k -> 2.2k; device jonnew:R_0402 -> jonnew:RN2X8_1506
- R57, R58: value 165k -> 2k
- R59: value 2.2k -> 10k; device jonnew:RN2X8_1506 -> jonnew:R_0402
- R60, R61: value 2.2k -> 3.48k; device jonnew:RN2X8_1506 -> jonnew:R_0402
- R62: value 2.2k -> 649k; device jonnew:RN2X8_1506 -> jonnew:R_0402
- R63: value 2k -> 0
- R64: value 2k -> 10k
- R66, R67: value 3.48k -> 10k
- R68: value 649k -> 10k
- R69: value 0 -> 2.2k
- R70: value 10k -> 15k
- R72, R74: value 10k -> 47k
- R75: value 2.2k -> 4.7k
- R76: value 15k -> 165k
- R77: value 4.7k -> 178k
- R78: value 43k -> 10k
- R80: value 43k -> 73.2k
- R81: value 4.7k -> 73.2k
- U11: value DS90UB934-Q1 -> DS91M040; device jonnew:DS90UB934-Q1 -> jonnew:DS91M040_WQFN32
- U12: value DS91M040 -> AD5766BCPZ-RL7; device jonnew:DS91M040_WQFN32 -> jonnew:AD5767BCBZ-RL7_QFN
- U13: value AD5766BCPZ-RL7 -> MCP47FEB02A0-E/ST; device jonnew:AD5767BCBZ-RL7_QFN -> jonnew:MCP47FEBX2
- U14: value MCP47FEB02A0-E/ST -> LM4132AMF-2.5/NOPBCT-ND; device jonnew:MCP47FEBX2 -> jonnew:VREF_EN_LM4132
- U15: value LM4132AMF-2.5/NOPBCT-ND -> AD7617BSTZ; device jonnew:VREF_EN_LM4132 -> jonnew:AD7617BSTZ
- U16: value AD7617BSTZ -> AD5142BCPZ10; device jonnew:AD7617BSTZ -> jonnew:AD51X2_QFN
- U17: value AD5142BCPZ10 -> LTM4622A; device jonnew:AD51X2_QFN -> jonnew:LTM4622_BGA
- U19: value TPS62293DRV -> TPS7A49; device jonnew:TPS6229X_WSON -> jonnew:TPS7AXX_PVSON
- U21: value TPS7A49 -> TPS7A30
- U22: value TPS7A30 -> 24AA64ST; device jonnew:TPS7AXX_PVSON -> jonnew:24AA64ST
- U23: value 24AA64ST -> LTM8049_BGA; device jonnew:24AA64ST -> jonnew:LTM8049_BGA
- U24: value LTM8049_BGA -> TPS62061DSGT; device jonnew:LTM8049_BGA -> jonnew:TPS6206X
- U4: value LTC2875_DFN -> ADCMP600; device jonnew:LTC2875_DFN -> jonnew:COMPARITOR_ADCMP600
- U6: value ADCMP600 -> DG1412E; device jonnew:COMPARITOR_ADCMP600 -> jonnew:DG141XE_QUAD_SPST_QFN
- U9: value DG1412E -> DS90UB934-Q1; device jonnew:DG141XE_QUAD_SPST_QFN -> jonnew:DS90UB934-Q1
Connections:
- removed net CAN_N: R27.2, SJ1.2, U4.CANL
- removed net CAN_P: R26.2, SJ2.2, U4.CANH
- removed net CAN_RX: J10G$5.HA02_N, U4.RXD
- removed net CAN_TX: J10G$5.HA02_P, U4.TXD
- removed net DEBUG0: J10G$2.LA06_P, J8.2
- removed net DEBUG1: J10G$2.LA06_N, J8.4
- removed net DEBUG2: J10G$2.LA09_P, J8.6
- removed net DEBUG3: J10G$2.LA10_P, J8.8
- removed net DEBUG4: J10G$2.LA09_N, J8.10
- removed net DEBUG5: J10G$2.LA10_N, J8.12
- removed net DEBUG6: J10G$2.LA14_P, J8.14
- removed net DEBUG7: J10G$2.LA14_N, J8.16
- removed net LVDS_DIN2_N/CAN_P: J7.2, SJ2.COM
- removed net LVDS_DIN2_P/CAN_N: J7.15, SJ1.COM
- removed net N$13: R33.2, U4.RS
- removed net N$36: D3.C, R3.1
- removed net N$41: C5.1, R26.1, R27.1, U4.SPLIT
- removed net N$57: D1.A, R1.1
- removed net N$66: D2.A, R2.1
- new net FMC_PG: J9G$2.PG_C2M, J9G$3.PG_M2C
- new net N$51: C129.2, J9G$6.STANDOFF_B
- new net N$52: C128.2, J9G$6.STANDOFF_A
- net !ADC_CS: now also J9G$4.LA07_P, U15.!CS; no longer J10G$4.LA07_P, U16.!CS
- net !ADC_RESET: now also J9G$3.HA08_P, R66.2; no longer J10G$3.HA08_P, R72.2
- net !DAC_CS: now also J9G$5.HA14_N, U12.!CS; no longer J10G$5.HA14_N, U13.!CS
- net !DAC_RESET: now also J9G$3.HA12_N, U12.!RESET; no longer J10G$3.HA12_N, U13.!RESET
- net !LINK_PWR_ADJ_CS: now also J9G$3.HB20_N, U16.!CS; no longer J10G$3.HB20_N, U17.!CS
- net !LINK_PWR_ADJ_RESET: now also J9G$3.HB21_N, U16.!RESET; no longer J10G$3.HB21_N, U17.!RESET
- net $N1: now also D5.COMM, R12.2, R2.2, R24.1, R6.2, R8.2; no longer D8.COMM, R11.2, R15.2, R29.1, R5.2, R9.2
- net $N2: now also D3.COMM; no longer D6.COMM
- net $N3: now also D4.COMM, R1.2, R11.2, R23.1, R5.2, R7.2; no longer D7.COMM, R10.2, R14.2, R28.1, R4.2, R8.2
- net +12V: now also C116.2, C135.2, J9G$2.12P0V1, J9G$2.12P0V2, R38.2, R39.2, U17.VIN; no longer C118.2, C130.2, J10G$2.12P0V1, J10G$2.12P0V2, R44.2, R45.2, U18.VIN
- net +13V_AN: now also C104.2, C105.2, C7.2, U12.AVDD, U6.V+; no longer C10.2, C106.2, C107.2, R2.2, U13.AVDD, U9.V+
- net +15V: now also C130.2, R76.1, U23.VOUT1P; no longer C131.2, R82.1, U24.VOUT1P
- net +1V8: now also C106.2, C86.2, C87.2, C91.2, C92.2, R19.1, R21.1, R34.1, R36.1, U24.FB, U9.VDD18; no longer C108.2, C88.2, C89.2, C93.2, C94.2, R22.1, R24.1, R40.1, R42.1, U11.VDD18, U19.FB
- net +3V3: now also C10.2, C111.2, C114.2, C117.2, C118.2, C22.1, C28.1, C32.1, C74.2, C78.2, C82.2, C89.2, C93.2, C96.2, J9G$3.VADJ@1, J9G$3.VADJ@2, J9G$4.VADJ@1, J9G$4.VADJ@2, J9G$5.VIO_B_M2C@1, J9G$5.VIO_B_M2C@2, R30.2, R31.2, R32.2, R33.2, R40.2, R43.2, R57.2, R58.2, R63.1, R64.1, R65.1, R78.2, R79.2, U11.VDD, U12.VLOGIC, U13.REFA, U13.VDD, U15.VDRIVE, U16.INDEP, U16.VDD, U16.VLOGIC, U23.RUN1, U23.RUN2, U23.VIN1, U23.VIN2, U24.AVIN, U24.EN, U24.MODE, U24.PVIN, U4G$2.V+, U9.OEN, U9.OSS_SEL; no longer C11.2, C115.2, C116.2, C119.2, C120.2, C24.1, C30.1, C34.1, C39.1, C76.2, C80.2, C84.2, C91.2, C95.2, C98.2, J10G$3.VADJ@1, J10G$3.VADJ@2, J10G$4.VADJ@1, J10G$4.VADJ@2, J10G$5.VIO_B_M2C@1, J10G$5.VIO_B_M2C@2, R36.2, R37.2, R38.2, R39.2, R46.2, R49.2, R63.2, R64.2, R70.1, R71.1, R75.1, R84.2, R85.2, U11.OEN, U11.OSS_SEL, U12.VDD, U13.VLOGIC, U14.REFA, U14.VDD, U16.VDRIVE, U17.INDEP, U17.VDD, U17.VLOGIC, U19.EN, U19.MODE, U19.VIN, U24.RUN1, U24.RUN2, U24.VIN1, U24.VIN2, U4.VCC, U6G$2.V+
- net +5V_AN: now also C107.2, C108.2, C59.2, C62.2, C69.2, C77.2, C81.1, C83.2, C84.2, C90.2, U12.AVCC, U14.EN, U14.VIN, U15.VCC; no longer C109.2, C110.2, C61.2, C64.2, C71.2, C79.2, C83.1, C86.2, C87.2, C92.2, R1.2, U13.AVCC, U15.EN, U15.VIN, U16.VCC
- net -13V_AN: now also C103.2, C17.2, C99.2, U12.AVSS, U6.V-; no longer C101.2, C105.2, C20.2, R3.2, U13.AVSS, U9.V-
- net -15V: now also C131.1, R77.1, U23.VOUT2N; no longer C132.1, R83.1, U24.VOUT2N
- net ADC_BUSY: now also J9G$5.HA11_P, U15.BUSY; no longer J10G$5.HA11_P, U16.BUSY
- net ADC_CONVST: now also J9G$5.HA10_P, U15.CONVST; no longer J10G$5.HA10_P, U16.CONVST
- net ADC_MISO_A: now also J9G$5.HA06_N, U15.DB12/SDOA; no longer J10G$5.HA06_N, U16.DB12/SDOA
- net ADC_MISO_B: now also J9G$5.HA07_N, U15.DB11/SDOB; no longer J10G$5.HA07_N, U16.DB11/SDOB
- net ADC_MOSI: now also J9G$5.HA06_P, U15.DB10/SDI; no longer J10G$5.HA06_P, U16.DB10/SDI
- net ADC_SCLK: now also J9G$5.HA11_N, U15.SCLK/!RD; no longer J10G$5.HA11_N, U16.SCLK/!RD
- net ADDR0: now also J9G$2.LA27_N, R78.1; no longer J10G$2.LA27_N, R84.1
- net ADDR1: now also J9G$2.LA27_P, R79.1; no longer J10G$2.LA27_P, R85.1
- net AGND: now also C100.1, C104.1, C108.1, C17.1, C59.1, C62.1, C69.1, C7.1, C77.1, C81.2, C83.1, C84.1, C88.1, C95.1, C99.1, R48.1, R53.C2, R53.C4, R53.C6, R53.C7, R54.C1, R54.C3, R54.C5, R54.C6, R54.C7, R54.C8, R55.C2, R55.C3, R55.C5, R55.C7, R56.C1, R56.C2, R56.C3, R56.C4, R56.C6, R56.C8, U12.AGND, U12.N0, U12.N1, U12.NIC, U14.GND, U15.AGND, U15.REFGND, U15.REFINOUTGND, U15.REGGND, U6.GND; no longer C10.1, C102.1, C106.1, C109.1, C110.1, C20.1, C61.1, C64.1, C71.1, C79.1, C83.2, C86.1, C87.1, C92.1, C97.1, D1.C, D2.C, D3.A, R54.1, R59.C2, R59.C4, R59.C6, R59.C7, R60.C1, R60.C3, R60.C5, R60.C6, R60.C7, R60.C8, R61.C2, R61.C3, R61.C5, R61.C7, R62.C1, R62.C2, R62.C3, R62.C4, R62.C6, R62.C8, U13.AGND, U13.N0, U13.N1, U13.NIC, U15.GND, U16.AGND, U16.REFGND, U16.REFINOUTGND, U16.REGGND, U9.GND
- net AIN_AOUT0: now also J9G$3.HA08_N, U8.IN1; no longer J10G$3.HA08_N, U9.IN1
- net AIN_AOUT1: now also J9G$2.LA05_P, U8.IN4; no longer J10G$2.LA05_P, U9.IN4
- net AIN_AOUT10: now also J9G$4.LA16_N, U6.IN4; no longer J10G$4.LA16_N, U7.IN4
- net AIN_AOUT11: now also J9G$4.LA15_P, U6.IN1; no longer J10G$4.LA15_P, U7.IN1
- net AIN_AOUT2: now also J9G$3.HA13_P, U8.IN3; no longer J10G$3.HA13_P, U9.IN3
- net AIN_AOUT3: now also J9G$4.LA04_P, U8.IN2; no longer J10G$4.LA04_P, U9.IN2
- net AIN_AOUT4: now also J9G$3.HA20_P, U7.IN1; no longer J10G$3.HA20_P, U8.IN1
- net AIN_AOUT5: now also J9G$5.HA07_P, U7.IN4; no longer J10G$5.HA07_P, U8.IN4
- net AIN_AOUT6: now also J9G$4.LA03_N, U7.IN3; no longer J10G$4.LA03_N, U8.IN3
- net AIN_AOUT7: now also J9G$3.HA15_N, U7.IN2; no longer J10G$3.HA15_N, U8.IN2
- net AIN_AOUT8: now also J9G$4.LA15_N, U6.IN3; no longer J10G$4.LA15_N, U7.IN3
- net AIN_AOUT9: now also J9G$5.HA18_P, U6.IN2; no longer J10G$5.HA18_P, U7.IN2
- net AIO_0: now also R53.C1, U8.D1; no longer R59.C1, U9.D1
- net AIO_1: now also R53.C3, U8.D4; no longer R59.C3, U9.D4
- net AIO_10: now also R55.C4, U6.D4; no longer R61.C4, U7.D4
- net AIO_11: now also R55.C1, U6.D1; no longer R61.C1, U7.D1
- net AIO_2: now also R53.C5, U8.D3; no longer R59.C5, U9.D3
- net AIO_3: now also R53.C8, U8.D2; no longer R59.C8, U9.D2
- net AIO_4: now also R54.C4, U7.D1; no longer R60.C4, U8.D1
- net AIO_5: now also R54.C2, U7.D4; no longer R60.C2, U8.D4
- net AIO_6: now also R56.C5, U7.D3; no longer R62.C5, U8.D3
- net AIO_7: now also R56.C7, U7.D2; no longer R62.C7, U8.D2
- net AIO_8: now also R55.C6, U6.D3; no longer R61.C6, U7.D3
- net AIO_9: now also R55.C8, U6.D2; no longer R61.C8, U7.D2
- net AOUT0: now also U12.VOUT0, U6.S1; no longer U13.VOUT0, U7.S1
- net AOUT1: now also U12.VOUT1, U6.S4; no longer U13.VOUT1, U7.S4
- net AOUT10: now also U12.VOUT10, U8.S4; no longer U13.VOUT10, U9.S4
- net AOUT11: now also U12.VOUT11, U8.S1; no longer U13.VOUT11, U9.S1
- net AOUT2: now also U12.VOUT2, U6.S3; no longer U13.VOUT2, U7.S3
- net AOUT3: now also U12.VOUT3, U6.S2; no longer U13.VOUT3, U7.S2
- net AOUT4: now also U12.VOUT4, U7.S1; no longer U13.VOUT4, U8.S1
- net AOUT5: now also U12.VOUT5, U7.S4; no longer U13.VOUT5, U8.S4
- net AOUT6: now also U12.VOUT6, U7.S2; no longer U13.VOUT6, U8.S2
- net AOUT7: now also U12.VOUT7, U7.S3; no longer U13.VOUT7, U8.S3
- net AOUT8: now also U12.VOUT8, U8.S3; no longer U13.VOUT8, U9.S3
- net AOUT9: now also U12.VOUT9, U8.S2; no longer U13.VOUT9, U9.S2
- net CLKIN0: now also J9G$2.LA17_N_CC, U4G$1.OUT; no longer J10G$2.LA17_N_CC, U5G$1.OUT
- net CLKIN1: now also J9G$3.HA20_N, U5G$1.OUT; no longer J10G$3.HA20_N, U6G$1.OUT
- net CLKIN_TERM0: now also J9G$5.HA21_P, R17.1; no longer J10G$5.HA21_P, R20.1
- net CLKIN_TERM1: now also J9G$5.HA17_N_CC, R18.1; no longer J10G$5.HA17_N_CC, R21.1
- net CLKIN_VBIAS_SCL: now also J9G$5.HA22_P, R58.1, U13.SCL; no longer J10G$5.HA22_P, R64.1, U14.SCL
- net CLKIN_VBIAS_SDA: now also J9G$5.HA21_N, R57.1, U13.SDA; no longer J10G$5.HA21_N, R63.1, U14.SDA
- net CLKOUT: now also J9G$2.LA17_P_CC; no longer J10G$2.LA17_P_CC
- net DAC_MISO: now also J9G$5.HA17_P_CC, U12.MISO; no longer J10G$5.HA17_P_CC, U13.MISO
- net DAC_MOSI: now also J9G$4.LA07_N, U12.MOSI; no longer J10G$4.LA07_N, U13.MOSI
- net DAC_MUX: now also U12.MUX_OUT; no longer U13.MUX_OUT
- net DAC_SCLK: now also J9G$5.HA14_P, U12.SCLK; no longer J10G$5.HA14_P, U13.SCLK
- net DES_A_D0: now also J9G$3.HB16_P, U10.ROUT0; no longer J10G$3.HB16_P, U11.ROUT0
- net DES_A_D1: now also J9G$5.HB14_N, U10.ROUT1; no longer J10G$5.HB14_N, U11.ROUT1
- net DES_A_D10: now also J9G$5.HB11_N, U10.ROUT10; no longer J10G$5.HB11_N, U11.ROUT10
- net DES_A_D11: now also J9G$5.HB10_P, U10.ROUT11; no longer J10G$5.HB10_P, U11.ROUT11
- net DES_A_D2: now also J9G$5.HB15_N, U10.ROUT2; no longer J10G$5.HB15_N, U11.ROUT2
- net DES_A_D3: now also J9G$5.HB14_P, U10.ROUT3; no longer J10G$5.HB14_P, U11.ROUT3
- net DES_A_D4: now also J9G$3.HB19_P, U10.ROUT4; no longer J10G$3.HB19_P, U11.ROUT4
- net DES_A_D5: now also J9G$5.HB15_P, U10.ROUT5; no longer J10G$5.HB15_P, U11.ROUT5
- net DES_A_D6: now also J9G$3.HB12_N, U10.ROUT6; no longer J10G$3.HB12_N, U11.ROUT6
- net DES_A_D7: now also J9G$3.HB13_N, U10.ROUT7; no longer J10G$3.HB13_N, U11.ROUT7
- net DES_A_D8: now also J9G$5.HB10_N, U10.ROUT8; no longer J10G$5.HB10_N, U11.ROUT8
- net DES_A_D9: now also J9G$3.HB12_P, U10.ROUT9; no longer J10G$3.HB12_P, U11.ROUT9
- net DES_A_GPIO0: now also J9G$5.HB18_N, U10.GPIO0; no longer J10G$5.HB18_N, U11.GPIO0
- net DES_A_GPIO1: now also J9G$5.HB17_P_CC, U10.GPIO1; no longer J10G$5.HB17_P_CC, U11.GPIO1
- net DES_A_GPIO2: now also J9G$5.HB18_P, U10.GPIO2; no longer J10G$5.HB18_P, U11.GPIO2
- net DES_A_GPIO3: now also J9G$3.HB19_N, R43.1, U10.GPIO3/INTB; no longer J10G$3.HB19_N, R49.1, U11.GPIO3/INTB
- net DES_A_HSYNC: now also J9G$3.HB13_P, U10.HSYNC; no longer J10G$3.HB13_P, U11.HSYNC
- net DES_A_LEDG: now also J9G$3.HB08_P, R47.2; no longer J10G$3.HB08_P, R53.2
- net DES_A_LOCK: now also J9G$3.HB09_P, R42.2, R50.2, U10.LOCK; no longer J10G$3.HB09_P, R48.2, R56.2, U11.LOCK
- net DES_A_PASS: now also J9G$5.HB07_N, R45.2, R52.2, U10.PASS; no longer J10G$5.HB07_N, R51.2, R58.2, U11.PASS
- net DES_A_PCLK: now also J9G$5.HB06_P_CC, U10.PCLK; no longer J10G$5.HB06_P_CC, U11.PCLK
- net DES_A_PDB: now also J9G$3.HB16_N, U10.PDB; no longer J10G$3.HB16_N, U11.PDB
- net DES_A_SCL: now also J9G$3.HB08_N, R31.1, U10.SCL; no longer J10G$3.HB08_N, R37.1, U11.SCL
- net DES_A_SDA\: now also J9G$3.HB09_N, R33.1, U10.SDA; no longer J10G$3.HB09_N, R39.1, U11.SDA
- net DES_A_VSYNC: now also J9G$5.HB11_P, U10.VSYNC; no longer J10G$5.HB11_P, U11.VSYNC
- net DES_B_D0: now also J9G$4.LA24_N, U9.ROUT0; no longer J10G$4.LA24_N, U10.ROUT0
- net DES_B_D1: now also J9G$4.LA24_P, U9.ROUT1; no longer J10G$4.LA24_P, U10.ROUT1
- net DES_B_D10: now also J9G$4.LA22_P, U9.ROUT10; no longer J10G$4.LA22_P, U10.ROUT10
- net DES_B_D11: now also J9G$2.LA23_P, U9.ROUT11; no longer J10G$2.LA23_P, U10.ROUT11
- net DES_B_D2: now also J9G$4.LA25_N, U9.ROUT2; no longer J10G$4.LA25_N, U10.ROUT2
- net DES_B_D3: now also J9G$4.LA25_P, U9.ROUT3; no longer J10G$4.LA25_P, U10.ROUT3
- net DES_B_D4: now also J9G$2.LA26_N, U9.ROUT4; no longer J10G$2.LA26_N, U10.ROUT4
- net DES_B_D5: now also J9G$2.LA26_P, U9.ROUT5; no longer J10G$2.LA26_P, U10.ROUT5
- net DES_B_D6: now also J9G$4.LA21_N, U9.ROUT6; no longer J10G$4.LA21_N, U10.ROUT6
- net DES_B_D7: now also J9G$4.LA22_N, U9.ROUT7; no longer J10G$4.LA22_N, U10.ROUT7
- net DES_B_D8: now also J9G$4.LA21_P, U9.ROUT8; no longer J10G$4.LA21_P, U10.ROUT8
- net DES_B_D9: now also J9G$2.LA23_N, U9.ROUT9; no longer J10G$2.LA23_N, U10.ROUT9
- net DES_B_GPIO0: now also J9G$4.LA28_N, U9.GPIO0; no longer J10G$4.LA28_N, U10.GPIO0
- net DES_B_GPIO1: now also J9G$4.LA29_N, U9.GPIO1; no longer J10G$4.LA29_N, U10.GPIO1
- net DES_B_GPIO2: now also J9G$4.LA28_P, U9.GPIO2; no longer J10G$4.LA28_P, U10.GPIO2
- net DES_B_GPIO3: now also J9G$4.LA29_P, R40.1, U9.GPIO3/INTB; no longer J10G$4.LA29_P, R46.1, U10.GPIO3/INTB
- net DES_B_HSYNC\: now also J9G$4.LA19_N, U9.HSYNC; no longer J10G$4.LA19_N, U10.HSYNC
- net DES_B_LEDG: now also J9G$4.LA20_P, R46.2; no longer J10G$4.LA20_P, R52.2
- net DES_B_LOCK: now also J9G$5.HA22_N, R41.2, R49.2, U9.LOCK; no longer J10G$5.HA22_N, R47.2, R55.2, U10.LOCK
- net DES_B_PASS: now also J9G$5.HA23_P, R44.2, R51.2, U9.PASS; no longer J10G$5.HA23_P, R50.2, R57.2, U10.PASS
- net DES_B_PCLK: now also J9G$2.LA18_P_CC, U9.PCLK; no longer J10G$2.LA18_P_CC, U10.PCLK
- net DES_B_PDB: now also J9G$4.LA31_P, U9.PDB; no longer J10G$4.LA31_P, U10.PDB
- net DES_B_SCL: now also J9G$4.LA20_N, R30.1, U9.SCL; no longer J10G$4.LA20_N, R36.1, U10.SCL
- net DES_B_SDA: now also J9G$4.LA19_P, R32.1, U9.SDA; no longer J10G$4.LA19_P, R38.1, U10.SDA
- net DES_B_VSYNC: now also J9G$5.HA23_N, U9.VSYNC; no longer J10G$5.HA23_N, U10.VSYNC
- net DI_VBIAS0: now also R15.1, U13.VOUT0; no longer R18.1, U14.VOUT0
- net DI_VBIAS1: now also R16.1, U13.VOUT1; no longer R19.1, U14.VOUT1
- net DOUTP_F_A: now also C45.2, D2.C, R4.2; no longer C47.2, D5.C, R7.2
- net DOUTP_F_B: now also C44.2, D1.C, R3.2; no longer C46.2, D4.C, R6.2
- net GND: now also C10.1, C102.1, C106.1, C109.1, C110.1, C115.2, C117.1, C122.2, C123.2, C125.1, C126.1, C13.2, C131.2, C132.1, C20.1, C22.2, C24.1, C28.2, C34.1, C40.1, C41.1, C46.1, C47.1, C5.1, C61.1, C64.1, C71.1, C79.1, C86.1, C87.1, C92.1, C97.1, D1.A, D2.A, D3.A, D7G$1.C, D7G$2.C, D7G$3.C, D8G$1.C, D8G$2.C, D8G$3.C, J9G$1.GND@1, J9G$1.GND@10, J9G$1.GND@11, J9G$1.GND@12, J9G$1.GND@13, J9G$1.GND@14, J9G$1.GND@15, J9G$1.GND@16, J9G$1.GND@17, J9G$1.GND@18, J9G$1.GND@19, J9G$1.GND@2, J9G$1.GND@20, J9G$1.GND@21, J9G$1.GND@22, J9G$1.GND@23, J9G$1.GND@24, J9G$1.GND@25, J9G$1.GND@26, J9G$1.GND@27, J9G$1.GND@28, J9G$1.GND@29, J9G$1.GND@3, J9G$1.GND@30, J9G$1.GND@31, J9G$1.GND@32, J9G$1.GND@33, J9G$1.GND@34, J9G$1.GND@35, J9G$1.GND@36, J9G$1.GND@37, J9G$1.GND@38, J9G$1.GND@39, J9G$1.GND@4, J9G$1.GND@40, J9G$1.GND@5, J9G$1.GND@6, J9G$1.GND@7, J9G$1.GND@8, J9G$1.GND@9, J9G$2.GA0, J9G$2.GA1, J9G$2.GND@1, J9G$2.GND@10, J9G$2.GND@11, J9G$2.GND@12, J9G$2.GND@13, J9G$2.GND@14, J9G$2.GND@15, J9G$2.GND@16, J9G$2.GND@17, J9G$2.GND@18, J9G$2.GND@19, J9G$2.GND@2, J9G$2.GND@20, J9G$2.GND@21, J9G$2.GND@23, J9G$2.GND@24, J9G$2.GND@25, J9G$2.GND@26, J9G$2.GND@27, J9G$2.GND@28, J9G$2.GND@29, J9G$2.GND@3, J9G$2.GND@30, J9G$2.GND@31, J9G$2.GND@33, J9G$2.GND@4, J9G$2.GND@5, J9G$2.GND@6, J9G$2.GND@7, J9G$2.GND@8, J9G$2.GND@9, J9G$3.GND@1, J9G$3.GND@10, J9G$3.GND@11, J9G$3.GND@12, J9G$3.GND@13, J9G$3.GND@14, J9G$3.GND@15, J9G$3.GND@16, J9G$3.GND@17, J9G$3.GND@18, J9G$3.GND@19, J9G$3.GND@2, J9G$3.GND@20, J9G$3.GND@21, J9G$3.GND@22, J9G$3.GND@23, J9G$3.GND@24, J9G$3.GND@25, J9G$3.GND@26, J9G$3.GND@27, J9G$3.GND@28, J9G$3.GND@29, J9G$3.GND@3, J9G$3.GND@4, J9G$3.GND@5, J9G$3.GND@6, J9G$3.GND@7, J9G$3.GND@8, J9G$3.GND@9, J9G$4.GND@1, J9G$4.GND@10, J9G$4.GND@11, J9G$4.GND@12, J9G$4.GND@13, J9G$4.GND@14, J9G$4.GND@15, J9G$4.GND@16, J9G$4.GND@17, J9G$4.GND@18, J9G$4.GND@19, J9G$4.GND@2, J9G$4.GND@20, J9G$4.GND@21, J9G$4.GND@22, J9G$4.GND@23, J9G$4.GND@24, J9G$4.GND@25, J9G$4.GND@26, J9G$4.GND@27, J9G$4.GND@28, J9G$4.GND@3, J9G$4.GND@4, J9G$4.GND@5, J9G$4.GND@6, J9G$4.GND@7, J9G$4.GND@8, J9G$4.GND@9, J9G$4.PRSNT_M2C_L, J9G$5.GND@1, J9G$5.GND@10, J9G$5.GND@11, J9G$5.GND@12, J9G$5.GND@13, J9G$5.GND@14, J9G$5.GND@15, J9G$5.GND@16, J9G$5.GND@17, J9G$5.GND@18, J9G$5.GND@19, J9G$5.GND@2, J9G$5.GND@20, J9G$5.GND@21, J9G$5.GND@22, J9G$5.GND@23, J9G$5.GND@24, J9G$5.GND@25, J9G$5.GND@26, J9G$5.GND@27, J9G$5.GND@28, J9G$5.GND@29, J9G$5.GND@3, J9G$5.GND@4, J9G$5.GND@5, J9G$5.GND@6, J9G$5.GND@7, J9G$5.GND@8, J9G$5.GND@9, R1.1, R13.1, R14.1, R2.1, R20.2, R22.2, R28.2, R29.2, R37.2, R48.2, R49.1, R50.1, R51.1, R52.1, R62.2, R67.2, R71.1, R73.1, R75.1, R80.2, R81.2, U12.DGND, U13.AVSS, U13.LAT/HVC, U15.CHSEL0, U15.CHSEL1, U15.CHSEL2, U15.DB0, U15.DB1, U15.DB13/OS0, U15.DB14/OS1, U15.DB15/OS2, U15.DB2, U15.DB3, U15.DB5/CRCEN, U15.DB6, U15.DB7, U15.DB8, U15.DB9, U15.DGND, U15.HW_RNGSEL0, U15.HW_RNGSEL1, U15.REGGNDD, U15.SEQEN, U15.WR!/BURST, U16.GND, U16.VSS, U16.W1, U16.W2, U17.SYNC/MODE, U19.NC, U19.PAD, U22.A0, U22.A1, U22.A2, U22.WP, U23.SYNC1, U23.VOUT1N, U23.VOUT2P, U24.AGND, U24.PGND, U4G$2.V-, U9.GND, U9.RES1, U9.RES2, U9.SEL; no longer C100.1, C104.1, C108.1, C115.1, C117.2, C122.1, C123.1, C125.2, C126.2, C13.1, C131.1, C132.2, C17.2, C22.1, C24.2, C28.1, C34.2, C38.1, C39.2, C44.1, C45.1, C5.2, C59.1, C62.1, C69.1, C7.1, C77.1, C81.1, C84.1, C88.1, C95.1, C99.1, D10G$1.C, D10G$2.C, D10G$3.C, D11G$1.C, D11G$2.C, D11G$3.C, D7.A, D8.A, D9.A, J10G$1.GND@1, J10G$1.GND@10, J10G$1.GND@11, J10G$1.GND@12, J10G$1.GND@13, J10G$1.GND@14, J10G$1.GND@15, J10G$1.GND@16, J10G$1.GND@17, J10G$1.GND@18, J10G$1.GND@19, J10G$1.GND@2, J10G$1.GND@20, J10G$1.GND@21, J10G$1.GND@22, J10G$1.GND@23, J10G$1.GND@24, J10G$1.GND@25, J10G$1.GND@26, J10G$1.GND@27, J10G$1.GND@28, J10G$1.GND@29, J10G$1.GND@3, J10G$1.GND@30, J10G$1.GND@31, J10G$1.GND@32, J10G$1.GND@33, J10G$1.GND@34, J10G$1.GND@35, J10G$1.GND@36, J10G$1.GND@37, J10G$1.GND@38, J10G$1.GND@39, J10G$1.GND@4, J10G$1.GND@40, J10G$1.GND@5, J10G$1.GND@6, J10G$1.GND@7, J10G$1.GND@8, J10G$1.GND@9, J10G$2.GA0, J10G$2.GA1, J10G$2.GND@1, J10G$2.GND@10, J10G$2.GND@11, J10G$2.GND@12, J10G$2.GND@13, J10G$2.GND@14, J10G$2.GND@15, J10G$2.GND@16, J10G$2.GND@17, J10G$2.GND@18, J10G$2.GND@19, J10G$2.GND@2, J10G$2.GND@20, J10G$2.GND@21, J10G$2.GND@23, J10G$2.GND@24, J10G$2.GND@25, J10G$2.GND@26, J10G$2.GND@27, J10G$2.GND@28, J10G$2.GND@29, J10G$2.GND@3, J10G$2.GND@30, J10G$2.GND@31, J10G$2.GND@33, J10G$2.GND@4, J10G$2.GND@5, J10G$2.GND@6, J10G$2.GND@7, J10G$2.GND@8, J10G$2.GND@9, J10G$3.GND@1, J10G$3.GND@10, J10G$3.GND@11, J10G$3.GND@12, J10G$3.GND@13, J10G$3.GND@14, J10G$3.GND@15, J10G$3.GND@16, J10G$3.GND@17, J10G$3.GND@18, J10G$3.GND@19, J10G$3.GND@21, J10G$3.GND@22, J10G$3.GND@23, J10G$3.GND@24, J10G$3.GND@25, J10G$3.GND@26, J10G$3.GND@27, J10G$3.GND@28, J10G$3.GND@29, J10G$3.GND@3, J10G$3.GND@4, J10G$3.GND@5, J10G$3.GND@6, J10G$3.GND@7, J10G$3.GND@8, J10G$3.GND@9, J10G$4.GND@1, J10G$4.GND@10, J10G$4.GND@11, J10G$4.GND@12, J10G$4.GND@13, J10G$4.GND@14, J10G$4.GND@15, J10G$4.GND@16, J10G$4.GND@17, J10G$4.GND@18, J10G$4.GND@19, J10G$4.GND@2, J10G$4.GND@20, J10G$4.GND@21, J10G$4.GND@22, J10G$4.GND@23, J10G$4.GND@24, J10G$4.GND@25, J10G$4.GND@26, J10G$4.GND@27, J10G$4.GND@28, J10G$4.GND@3, J10G$4.GND@4, J10G$4.GND@5, J10G$4.GND@6, J10G$4.GND@7, J10G$4.GND@8, J10G$4.GND@9, J10G$5.GND@1, J10G$5.GND@10, J10G$5.GND@11, J10G$5.GND@12, J10G$5.GND@13, J10G$5.GND@14, J10G$5.GND@15, J10G$5.GND@16, J10G$5.GND@17, J10G$5.GND@18, J10G$5.GND@19, J10G$5.GND@2, J10G$5.GND@20, J10G$5.GND@21, J10G$5.GND@22, J10G$5.GND@23, J10G$5.GND@24, J10G$5.GND@25, J10G$5.GND@26, J10G$5.GND@27, J10G$5.GND@28, J10G$5.GND@29, J10G$5.GND@3, J10G$5.GND@4, J10G$5.GND@5, J10G$5.GND@6, J10G$5.GND@7, J10G$5.GND@8, J10G$5.GND@9, J8.1, J8.11, J8.13, J8.15, J8.3, J8.5, J8.7, J8.9, R16.1, R17.1, R23.2, R25.2, R33.1, R34.2, R4.1, R41.2, R43.2, R5.1, R54.2, R55.1, R56.1, R57.1, R58.1, R73.2, R74.2, R77.1, R79.1, R81.1, R86.2, R87.2, U11.RES1, U11.RES2, U11.SEL, U12.GND, U13.DGND, U14.AVSS, U14.LAT/HVC, U16.CHSEL0, U16.CHSEL1, U16.CHSEL2, U16.DB0, U16.DB1, U16.DB13/OS0, U16.DB14/OS1, U16.DB15/OS2, U16.DB2, U16.DB3, U16.DB5/CRCEN, U16.DB6, U16.DB7, U16.DB8, U16.DB9, U16.DGND, U16.HW_RNGSEL0, U16.HW_RNGSEL1, U16.REGGNDD, U16.SEQEN, U16.WR!/BURST, U17.VSS, U17.W1, U17.W2, U18.GND, U18.SYNC/MODE, U22.NC, U22.PAD, U23.A0, U23.A1, U23.A2, U23.WP, U24.GND, U24.SYNC1, U24.VOUT1N, U24.VOUT2P, U4.GND, U6G$2.V-
- net LINK_A_PWR_EN: now also J9G$4.LA32_P, R68.1, U17.RUN2; no longer J10G$4.LA32_P, R74.1, U18.RUN2
- net LINK_B_PWR_EN: now also J9G$5.HB17_N_CC, R67.1, U17.RUN1; no longer J10G$5.HB17_N_CC, R73.1, U18.RUN1
- net LINK_PWR_ADJ_MISO: now also J9G$3.HB20_P, R69.2, U16.MISO; no longer J10G$3.HB20_P, R75.2, U17.MISO
- net LINK_PWR_ADJ_MOSI: now also J9G$3.HB21_P, U16.MOSI; no longer J10G$3.HB21_P, U17.MOSI
- net LINK_PWR_ADJ_SCLK: now also J9G$4.LA32_N, U16.SCLK; no longer J10G$4.LA32_N, U17.SCLK
- net LVDS_DIN0: now also J9G$5.CLK3_M2C_P; no longer J10G$5.CLK1_C2M_P
- net LVDS_DIN0_N: now also R25.1; no longer R30.1
- net LVDS_DIN0_P: now also R25.2; no longer R30.2
- net LVDS_DIN1: now also J9G$4.CLK0_M2C_N; no longer J10G$4.CLK0_M2C_N
- net LVDS_DIN1_N: now also R26.1; no longer R31.1
- net LVDS_DIN1_P: now also R26.2; no longer R31.2
- net LVDS_DIN2: now also J9G$4.CLK0_M2C_P; no longer J10G$4.CLK0_M2C_P
- net LVDS_DIN2_N: now also J7.2, R27.1; no longer R32.1, SJ2.1
- net LVDS_DIN2_P: now also J7.15, R27.2; no longer R32.2, SJ1.1
- net LVDS_DOUT0: now also J9G$5.CLK3_M2C_N; no longer J10G$5.CLK1_C2M_N
- net LVDS_DOUT1: now also J9G$5.CLK2_M2C_P; no longer J10G$5.CLK1_M2C_P
- net MLDVS_EN: now also J9G$4.LA02_N, U11.MDE; no longer J10G$4.LA02_N, U12.MDE
- net MLDVS_RO0: now also J9G$4.CLK1_M2C_P, U11.RO0; no longer J10G$4.CLK0_C2M_P, U12.RO0
- net MLDVS_RO1: now also J9G$3.HA01_N_CC, U11.RO1; no longer J10G$3.HA01_N_CC, U12.RO1
- net MLDVS_RO2: now also J9G$4.LA00_N_CC, U11.RO2; no longer J10G$4.LA00_N_CC, U12.RO2
- net MLDVS_RO3: now also J9G$3.HA00_P_CC, U11.RO3; no longer J10G$3.HA00_P_CC, U12.RO3
- net MLVDS_CLK_0_N: now also U11.B0; no longer U12.B0
- net MLVDS_CLK_0_P: now also U11.A0; no longer U12.A0
- net MLVDS_CLK_1_N: now also U11.B1; no longer U12.B1
- net MLVDS_CLK_1_P: now also U11.A1; no longer U12.A1
- net MLVDS_CLK_2_N: now also U11.B2; no longer U12.B2
- net MLVDS_CLK_2_P: now also U11.A2; no longer U12.A2
- net MLVDS_CLK_3_N: now also U11.B3; no longer U12.B3
- net MLVDS_CLK_3_P: now also U11.A3; no longer U12.A3
- net MLVDS_DE_!RE0: now also J9G$3.HA04_P, U11.!RE0, U11.DE0; no longer J10G$3.HA04_P, U12.!RE0, U12.DE0
- net MLVDS_DE_!RE1: now also J9G$3.HA05_N, U11.!RE1, U11.DE1; no longer J10G$3.HA05_N, U12.!RE1, U12.DE1
- net MLVDS_DE_!RE2: now also J9G$4.LA02_P, U11.!RE2, U11.DE2; no longer J10G$4.LA02_P, U12.!RE2, U12.DE2
- net MLVDS_DE_!RE3: now also J9G$3.HA04_N, U11.!RE3, U11.DE3; no longer J10G$3.HA04_N, U12.!RE3, U12.DE3
- net MLVDS_DI0: now also J9G$4.CLK1_M2C_N, U11.DI0; no longer J10G$4.CLK0_C2M_N, U12.DI0
- net MLVDS_DI1: now also J9G$3.HA01_P_CC, U11.DI1; no longer J10G$3.HA01_P_CC, U12.DI1
- net MLVDS_DI2: now also J9G$4.LA00_P_CC, U11.DI2; no longer J10G$4.LA00_P_CC, U12.DI2
- net MLVDS_DI3: now also J9G$3.HA00_N_CC, U11.DI3; no longer J10G$3.HA00_N_CC, U12.DI3
- net N$1: now also U24.SW; no longer U19.SW
- net N$10: now also R60.1, U17.FB1; no longer R66.1, U18.FB1
- net N$100: now also R34.2, R35.1, U9.IDX; no longer R40.2, R41.1, U10.IDX
- net N$118: now also D7G$1.A, R41.1; no longer D10G$1.A, R47.1
- net N$119: now also D7G$2.A, R44.1; no longer D10G$2.A, R50.1
- net N$12: now also C112.2, U17.TRACK/SS1; no longer C114.2, U18.TRACK/SS1
- net N$122: now also R60.2, U16.A1; no longer R66.2, U17.A1
- net N$123: now also R61.2, U16.A2; no longer R67.2, U17.A2
- net N$145: now also R62.1, U17.FREQ; no longer R68.1, U18.FREQ
- net N$15: now also C125.2, U19.EN, U19.IN; no longer C127.2, U20.EN, U20.IN
- net N$16: now also D8G$3.A, R47.1; no longer D11G$3.A, R53.1
- net N$17: now also R80.1, U23.RT1; no longer R86.1, U24.RT1
- net N$18: now also C13.1, R15.2, U4G$1.-IN; no longer C14.1, R18.2, U5G$1.-IN
- net N$19: now also R24.2, U5G$1.+IN; no longer R29.2, U6G$1.+IN
- net N$2: now also R11.1, R5.1, R7.1; no longer R10.1, R14.1, R8.1
- net N$20: now also C14.1, R16.2, U5G$1.-IN; no longer C15.1, R19.2, U6G$1.-IN
- net N$200: now also C56.2, C61.2, C66.2, C73.2, U10.VDDIO; no longer C58.2, C63.2, C68.2, C75.2, U11.VDDIO
- net N$21: now also R10.2, R4.1; no longer R13.2, R7.1
- net N$22: now also C16.1, C6.2, R10.1; no longer C17.1, C7.2, R13.1
- net N$23: now also R55.1, U15.V3B; no longer R61.1, U16.V3B
- net N$24: now also C15.1, C5.2, R9.1; no longer C16.1, C6.2, R12.1
- net N$25: now also R77.2, U23.FBX2; no longer R83.2, U24.FBX2
- net N$26: now also D7G$3.A, R46.1; no longer D10G$3.A, R52.1
- net N$27: now also C45.1, U10.RIN0+; no longer C47.1, U11.RIN0+
- net N$28: now also C39.1, U10.RIN0-; no longer C41.1, U11.RIN0-
- net N$29: now also R76.2, U23.FBX1; no longer R82.2, U24.FBX1
- net N$3: now also R23.2, U4G$1.+IN; no longer R28.2, U5G$1.+IN
- net N$30: now also C36.2, C42.2, C47.2, U10.VDD11_D; no longer C37.2, C44.2, C49.2, U11.VDD11_D
- net N$31: now also C37.2, C43.2, U10.VDD11_DVP; no longer C38.2, C45.2, U11.VDD11_DVP
- net N$32: now also C39.2, R29.1; no longer C41.2, R35.1
- net N$33: now also C122.1, U19.NR/SS; no longer C124.1, U20.NR/SS
- net N$34: now also R14.2, R18.2; no longer R17.2, R21.2
- net N$35: now also U23.CLKOUT1, U23.SYNC2; no longer U24.CLKOUT1, U24.SYNC2
- net N$37: now also R13.2, R17.2; no longer R16.2, R20.2
- net N$38: now also C44.1, U9.RIN0+; no longer C46.1, U10.RIN0+
- net N$39: now also R55.2, U15.V3BGND; no longer R61.2, U16.V3BGND
- net N$4: now also R3.1, R9.2; no longer R12.2, R6.1
- net N$40: now also R70.1, R71.2, U19.FB; no longer R76.1, R77.2, U20.FB
- net N$402: now also U10.BISTEN; no longer U11.BISTEN
- net N$403: now also R21.2, R22.1, U10.MODE; no longer R24.2, R25.1, U11.MODE
- net N$404: now also R36.2, R37.1, U10.IDX; no longer R42.2, R43.1, U11.IDX
- net N$42: now also C126.2, U20.EN, U20.IN; no longer C128.2, U21.EN, U21.IN
- net N$43: now also C123.1, U20.NR/SS; no longer C125.1, U21.NR/SS
- net N$45: now also C68.2, C76.2, C80.2, U10.VDD11_FPD; no longer C70.2, C78.2, C82.2, U11.VDD11_FPD
- net N$46: now also C115.1, R66.1, U15.!RESET; no longer C117.1, R72.1, U16.!RESET
- net N$47: now also C55.2, C60.2, C64.2, C71.2, U9.VDDIO; no longer C57.2, C62.2, C66.2, C73.2, U10.VDDIO
- net N$48: now also C34.2, C40.2, C46.2, U9.VDD11_D; no longer C35.2, C42.2, C48.2, U10.VDD11_D
- net N$49: now also C35.2, C41.2, U9.VDD11_DVP; no longer C36.2, C43.2, U10.VDD11_DVP
- net N$5: now also R61.1, U17.FB2; no longer R67.1, U18.FB2
- net N$50: now also C67.2, C75.2, C79.2, U9.VDD11_FPD; no longer C69.2, C77.2, C81.2, U10.VDD11_FPD
- net N$500: now also C119.2, R70.2, U19.OUT; no longer C121.2, R76.2, U20.OUT
- net N$501: now also C120.2, R72.2, U20.OUT; no longer C122.2, R78.2, U21.OUT
- net N$502: now also C121.2, R74.2, U21.OUT; no longer C123.2, R80.2, U22.OUT
- net N$506: now also C100.2, R59.1, U15.REFINOUT; no longer C102.2, R65.1, U16.REFINOUT
- net N$53: now also D8G$1.A, R42.1; no longer D11G$1.A, R48.1
- net N$54: now also D8G$2.A, R45.1; no longer D11G$2.A, R51.1
- net N$55: now also C38.1, U9.RIN0-; no longer C40.1, U10.RIN0-
- net N$56: now also R72.1, R73.2, U20.FB; no longer R78.1, R79.2, U21.FB
- net N$58: now also C127.2, U21.EN, U21.IN; no longer C129.2, U22.EN, U22.IN
- net N$59: now also C124.1, U21.NR/SS; no longer C126.1, U22.NR/SS
- net N$60: now also R74.1, R75.2, U21.FB; no longer R80.1, R81.2, U22.FB
- net N$603: now also U9.BISTEN; no longer U10.BISTEN
- net N$604: now also R19.2, R20.1, U9.MODE; no longer R22.2, R23.1, U10.MODE
- net N$61: now also R65.2, U15.DB4/!SER1WR; no longer R71.2, U16.DB4/!SER1WR
- net N$62: now also R53.1, U15.V0A; no longer R59.1, U16.V0A
- net N$63: now also R64.2, U15.SER/!PAR; no longer R70.2, U16.SER/!PAR
- net N$64: now also C95.2, U15.REFCAP; no longer C97.2, U16.REFCAP
- net N$65: now also R53.2, U15.V0AGND; no longer R59.2, U16.V0AGND
- net N$67: now also C109.2, U15.REGCAPD; no longer C111.2, U16.REGCAPD
- net N$68: now also R55.8, U15.V0B; no longer R61.8, U16.V0B
- net N$69: now also C101.2, U15.REGCAP; no longer C103.2, U16.REGCAP
- net N$7: now also R12.1, R6.1, R8.1; no longer R11.1, R15.1, R9.1
- net N$71: now also R63.2, U15.REFSEL; no longer R69.2, U16.REFSEL
- net N$72: now also R56.7, U15.V4B; no longer R62.7, U16.V4B
- net N$73: now also R56.1, U15.V7BGND; no longer R62.1, U16.V7BGND
- net N$74: now also R55.7, U15.V0BGND; no longer R61.7, U16.V0BGND
- net N$75: now also R55.6, U15.V1B; no longer R61.6, U16.V1B
- net N$76: now also R55.5, U15.V1BGND; no longer R61.5, U16.V1BGND
- net N$77: now also R55.4, U15.V2B; no longer R61.4, U16.V2B
- net N$78: now also R55.3, U15.V2BGND; no longer R61.3, U16.V2BGND
- net N$79: now also R53.3, U15.V1A; no longer R59.3, U16.V1A
- net N$8: now also C110.2, U17.TRACK/SS2; no longer C112.2, U18.TRACK/SS2
- net N$80: now also R53.4, U15.V1AGND; no longer R59.4, U16.V1AGND
- net N$81: now also R53.5, U15.V2A; no longer R59.5, U16.V2A
- net N$82: now also R53.6, U15.V2AGND; no longer R59.6, U16.V2AGND
- net N$83: now also R53.8, U15.V3A; no longer R59.8, U16.V3A
- net N$84: now also R53.7, U15.V3AGND; no longer R59.7, U16.V3AGND
- net N$85: now also R54.2, U15.V4A; no longer R60.2, U16.V4A
- net N$86: now also R54.1, U15.V4AGND; no longer R60.1, U16.V4AGND
- net N$87: now also R54.4, U15.V5A; no longer R60.4, U16.V5A
- net N$88: now also R54.3, U15.V5AGND; no longer R60.3, U16.V5AGND
- net N$89: now also R54.5, U15.V6A; no longer R60.5, U16.V6A
- net N$9: now also R81.1, U23.RT2; no longer R87.1, U24.RT2
- net N$90: now also R54.6, U15.V6AGND; no longer R60.6, U16.V6AGND
- net N$91: now also R54.7, U15.V7A; no longer R60.7, U16.V7A
- net N$92: now also R54.8, U15.V7AGND; no longer R60.8, U16.V7AGND
- net N$93: now also C38.2, R28.1; no longer C40.2, R34.1
- net N$94: now also R56.8, U15.V4BGND; no longer R62.8, U16.V4BGND
- net N$95: now also R56.5, U15.V5B; no longer R62.5, U16.V5B
- net N$96: now also R56.6, U15.V5BGND; no longer R62.6, U16.V5BGND
- net N$97: now also R56.4, U15.V6B; no longer R62.4, U16.V6B
- net N$98: now also R56.3, U15.V6BGND; no longer R62.3, U16.V6BGND
- net N$99: now also R56.2, U15.V7B; no longer R62.2, U16.V7B
- net SCL: now also J9G$2.SCL, U22.SCL; no longer J10G$2.SCL, U23.SCL
- net SDA: now also J9G$2.SDA, U22.SDA; no longer J10G$2.SDA, U23.SDA
- net TDI-TDO: now also J9G$2.TDI, J9G$2.TDO; no longer J10G$2.TDI, J10G$2.TDO
- net VAUX: now also C132.2, J9G$2.3P3VAUX, U22.VCC; no longer C135.2, J10G$2.3P3VAUX, U23.VCC
- net VDD_FPDX_A: now also C12.2, C21.2, C25.2, U10.VDD18_FPD0, U10.VDD18_FPD1; no longer C13.2, C22.2, C26.2, U11.VDD18_FPD0, U11.VDD18_FPD1
- net VDD_FPDX_B: now also C11.2, C20.2, C24.2, U9.VDD18_FPD0, U9.VDD18_FPD1; no longer C12.2, C21.2, C25.2, U10.VDD18_FPD0, U10.VDD18_FPD1
- net VDD_PX_A: now also C49.2, C54.2, C58.2, C65.2, C72.2, U10.VDD18_P0, U10.VDD18_P1; no longer C53.2, C56.2, C60.2, C67.2, C74.2, U11.VDD18_P0, U11.VDD18_P1
- net VDD_PX_B: now also C48.2, C53.2, C57.2, C63.2, C70.2, U9.VDD18_P0, U9.VDD18_P1; no longer C52.2, C55.2, C59.2, C65.2, C72.2, U10.VDD18_P0, U10.VDD18_P1
- net VLINK_A: now also C27.2, C31.1, C94.2, C97.2, U17.VOUT2; no longer C28.2, C32.1, C96.2, C99.2, U18.VOUT2
- net VLINK_B: now also C102.2, C26.2, C30.1, C98.2, U17.VOUT1; no longer C100.2, C104.2, C27.2, C31.1, U18.VOUT1
- net VREF: now also C88.2, R59.2, U12.VREF, U14.VOUT; no longer C90.2, R65.2, U13.VREF, U15.VOUT
- net V_PROTECT: now also C52.2, D3.C, D4.C, D5.C, R38.1, R39.1; no longer C54.2, D7.C, D8.C, D9.C, R44.1, R45.1
Other:
- note added: "NB: Required by FMC standard. Other option is to directly connect to front bezel"
- note removed: "DEBUG"
- note removed: "NB: Rs set to allow up to 4 Mbps."
- moved on the sheet: C10, C100, C101, C102, C103, C104, C105, C106, C107, C108, C109, C11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
