File: fmc-host/fmc-host.sch (EAGLE design)
At the start: 307 parts, among them J1 SMA002, J2 SMA002, J3 SMA002, J4 SMA002, J5 SMA002, J6 ESHF-105-01-L-D-SM-K-TR, J7 12226-8250-00FR, J8 FMC_SINGLE_WIDTH_MODULE, J9 ASP-134488-01, Q1 SI1012R, Q2 SI1012R, U1 SN74LVC2G34DCKR, U10 DS90UB934-Q1, U11 DS91M040, U12 AD5766BCPZ-RL7, U13 MCP47FEB02A0-E/ST, U14 LM4132AMF-2.5/NOPBCT-ND, U15 AD7617BSTZ, U16 AD5142BCPZ10, U17 LTM4622A, U19 TPS7A49, U2 SN65LVDS9638DGN, U20 TPS7A49, U21 TPS7A30, U22 24AA64ST, U23 LTM8049_BGA, U24 TPS62061DSGT, U3 FIN1032MTCX, U4 ADCMP600, U5 ADCMP600, U6 DG1412E, U7 DG1412E, U8 DG1412E, U9 DS90UB934-Q1, X2 OE-LOGO_7X5

Commit message: Revision 1.6
- The major change here is that I've swapped the vertical MVLVDS sync
header for a through-hole right-angle version that is much more
amenable to daisy chain connections when the card is in a PCIe slot.
- Deleted some obsolete, hard to maintain files
- Deleted some obsolete datasheets
Parts:
- J6: value ESHF-105-01-L-D-SM-K-TR -> FTSH-105-01-F-D-RA-K; device jonnew:PINHD-2X5_ESHF-SM -> jonnew:PINHD-2X5_FTSH
Connections:
- net MLDVS_RO2 renamed MLVDS_RO2
- removed net MLDVS_EN: J9G$4.LA02_N, U11.MDE
- removed net MLDVS_RO0: J9G$4.CLK1_M2C_P, U11.RO0
- removed net MLDVS_RO1: J9G$3.HA01_N_CC, U11.RO1
- removed net MLDVS_RO3: J9G$3.HA00_P_CC, U11.RO3
- new net MLVDS_EN: J9G$3.HA04_N, U11.MDE
- new net MLVDS_RO0: J9G$3.HA00_P_CC, U11.RO0
- new net MLVDS_RO1: J9G$4.LA00_P_CC, U11.RO1
- new net MLVDS_RO3: J9G$4.CLK1_M2C_P, U11.RO3
- net MLVDS_CLK_0_N: now also J6.10; no longer J6.9
- net MLVDS_CLK_0_P: now also J6.9; no longer J6.10
- net MLVDS_CLK_1_N: now also J6.8; no longer J6.7
- net MLVDS_CLK_1_P: now also J6.7; no longer J6.8
- net MLVDS_CLK_2_N: now also J6.4; no longer J6.3
- net MLVDS_CLK_2_P: now also J6.3; no longer J6.4
- net MLVDS_CLK_3_N: now also J6.2; no longer J6.1
- net MLVDS_CLK_3_P: now also J6.1; no longer J6.2
- net MLVDS_DE_!RE3: now also J9G$4.LA02_N; no longer J9G$3.HA04_N
- net MLVDS_DI0: now also J9G$3.HA00_N_CC; no longer J9G$4.CLK1_M2C_N
- net MLVDS_DI2: now also J9G$3.HA01_N_CC; no longer J9G$4.LA00_P_CC
- net MLVDS_DI3: now also J9G$4.CLK1_M2C_N; no longer J9G$3.HA00_N_CC
Other:
- note added: "CLOCK IO"
- note added: "DES. CORE POWER"
- note added: "FMC MEZZANINE"
- note added: "NB: All IO to to CC Pin or better"
- note added: "SYNC. TRIG."
- note removed: "CLK/TRIGGER I/0"
- note removed: "DES CORE POWER"
- note removed: "FMC"
- note removed: "INTERNAL CLK/TRIG"
- note removed: "NB: TO CC Pin"
- moved on the sheet: C102, C110, C111, C112, C113, C116, C94, C97, C98, J6, J7, R60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

Commit message: Revision F ready for fabrication feedback
- Replaced QFN AD5142 with TSSOP package, which is available
- Added ground pours to all layers
- Used thermals on top and bottom to improve solderability
Parts:
- removed D7, D8: APFA3011-AK13/F, jonnew:LED_3X_SMD-6
- added J10: BM08B-SURS-TF, jonnew:PINHD-1X8_SURS-TF
- C133, C136: value 47uF -> 33uF; device jonnew:C_1210 -> jonnew:C-POL_1411-VISHAY-B
- U16: device jonnew:AD51X2_QFN -> jonnew:AD51X2_TSSOP
Connections:
- removed net DES_A_LEDG: J9G$3.HB08_P, R47.2
- removed net DES_B_LEDG: J9G$4.LA20_P, R46.2
- removed net N$118: D7G$1.A, R41.1
- removed net N$119: D7G$2.A, R44.1
- removed net N$16: D8G$3.A, R47.1
- removed net N$26: D7G$3.A, R46.1
- removed net N$53: D8G$1.A, R42.1
- new net N$101: J10.4, R45.1
- new net N$102: J10.3, R46.1
- new net N$103: J10.1, R44.1
- new net N$57: J10.7, R47.1
- new net N$66: J10.8, R41.1
- new net PORT_A_BLUE: J9G$4.LA16_P, R41.2
- new net PORT_A_GREEN: J9G$5.HA18_P, R47.2
- new net PORT_A_RED: J9G$4.LA11_N, R42.1
- new net PORT_B_BLUE: J9G$4.LA11_P, R45.2
- new net PORT_B_GREEN: J9G$4.LA12_P, R46.2
- new net PORT_B_RED: J9G$4.LA08_N, R44.2
- net +12V: now also C133.+; no longer C133.2
- net +3V3: now also C136.+; no longer C136.2
- net AIN_AOUT9: now also J9G$5.HA18_N; no longer J9G$5.HA18_P
- net DES_A_LOCK: no longer R42.2
- net DES_A_PASS: no longer R45.2
- net DES_B_LOCK: no longer R41.2
- net DES_B_PASS: no longer R44.2
- net GND: now also C133.-, C136.-, J10.2, J10.6; no longer C133.1, C136.1, D7G$1.C, D7G$2.C, D7G$3.C, D8G$1.C, D8G$2.C, D8G$3.C
- net N$54: now also J10.5, R42.2; no longer D8G$2.A, R45.1
Other:
- note added: "PANEL RGB"
- moved on the sheet: C133, C136, R41, R42, R44, R45, R46, R47, U16
