File: pcb/fmc-host.kicad_pcb (KiCad board)
At the start: 6 copper layers, 76.5 x 339.8 mm, 310 parts, among them J1 SMA002, J10 BM08B-SURS-TF, J2 SMA002, J3 SMA002, J4 SMA002, J5 SMA002, J6 FTSH-105-01-F-D-RA-K, J7 12226-8250-00FR, J8 FMC_SINGLE_WIDTH_MODULE, J9 ASP-134488-01, Q1 SI1012R, Q2 SI1012R, U1 SN74LVC2G34DCKR, U10 DS90UB934-Q1, U11 DS91M040, U12 AD5766BCPZ-RL7, U13 MCP47FEB02A0-E/ST, U14 LM4132AMF-2.5/NOPBCT-ND, U15 AD7616BSTZ, U16 AD5142BCPZ10, U17 LTM4622A, U18 D3V3XA4B10LP, U19 TPS7A49, U2 SN65LVDS9638DGN, U20 TPS7A49, U21 TPS7A30, U22 24ST, U23 LTM8049_BGA, U24 TPS62061DSGT, U25 D3V3XA4B10LP, U26 D3V3XA4B10LP, U3 FIN1032MTCX, U4 ADCMP600, U5 ADCMP600, U6 DG1412E, U7 DG1412E, U8 DG1412E, U9 DS90UB934-Q1, X2 OE-LOGO_7X5

Commit message: Updated OEPS PN.
Added OEPS PN to all components.
The cross-check between BOM and PNP files failed due to TP (test points) attributes.
Fixed TP attributes.
Added .history/ to .gitignore to remove KiCAD history files.
Parts:
- D1, D2: value SESD0402X1UN-0020-090 -> SESD0402X1UN-0030-088
- D6: value KDZ4.3B -> KDZVTR4.3B
- J1, J2, J3, J4, J5: value SMA002 -> 6-1634010-0
- L5, L6: value SRNxx-101M -> SRN6045TA-101M
- U14: value LM4132AMF-2.5/NOPBCT-ND -> LM4132AMF-2.5/NOPB
- U16: value AD5142BCPZ10 -> AD5142BRUZ10
- U22: value 24ST -> 24AA64-I/ST
- U23: value LTM8049_BGA -> LTM8049IY#PBF
Changed lines of the file:
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@@
 			)
 		)
-		(property "Value" "LTM8049_BGA"
+		(property "Value" "LTM8049IY#PBF"
 			(at -4.4 -7.9 270)
 			(unlocked yes)
@@
 			)
 		)
-		(property "old description" "#N/A"
+		(property "old description" "DIODE:   RF DIODE PIN 150V 250MW   [BAR66E6327HTSA1] [PG-SOT23]"
 			(at 0 0 90)
 			(unlocked yes)
@@
 			)
 		)
-		(property "Value" "SRNxx-101M"
+		(property "Value" "SRN6045TA-101M"
 			(at -3 4 270)
 			(unlocked yes)
@@
 			)
 		)
-		(property "Value" "SMA002"
+		(property "Value" "6-1634010-0"
 			(at 2.5 1.5 90)
 			(unlocked yes)
@@
 			)
 		)
-		(property "Value" "SRNxx-101M"
+		(property "Value" "SRN6045TA-101M"
 			(at -3 4 270)
 			(unlocked yes)
@@
 			)
 		)
-		(property "MPN" "-"
+		(property "MPN" "DNP"
 			(at 0 0 90)
 			(unlocked yes)
@@
 			)
 		)
-		(property "old description" ""
+		(property "old description" "DNP: Do Not Populate (DNI)"
 			(at 0 0 90)
 			(unlocked yes)
@@
 			)
 		)
-		(property "Value" "SESD0402X1UN-0020-090"
+		(property "Value" "SESD0402X1UN-0030-088"
 			(at -1.27 1.778 0)
 			(unlocked yes)
@@
 			)
 		)
-		(property "Value" "AD5142BCPZ10"
+		(property "Value" "AD5142BRUZ10"
 			(at -2.7572 4.1385 0)
 			(unlocked yes)
@@
 			)
 		)
-		(property "Value" "SMA002"
+		(property "Value" "6-1634010-0"
 			(at 2.5 1.5 90)
 			(unlocked yes)
@@
 			)
 		)
-		(property "old description" "#N/A"
+		(property "old description" "DIODE:   RF DIODE PIN 150V 250MW   [BAR66E6327HTSA1] [PG-SOT23]"
 			(at 0 0 180)
 			(unlocked yes)
@@
 			)
 		)
-		(property "Value" "SESD0402X1UN-0020-090"
+		(property "Value" "SESD0402X1UN-0030-088"
 			(at -1.27 1.778 0)
 			(unlocked yes)
@@
 			)
 		)
-		(property "Value" "KDZ4.3B"
+		(property "Value" "KDZVTR4.3B"
 			(at -2.54 2.54 270)
 			(unlocked yes)
@@
 			)
 		)
-		(property "old description" "#N/A"
+		(property "old description" "DIODE:   RF DIODE PIN 150V 250MW   [BAR66E6327HTSA1] [PG-SOT23]"
 			(at 0 0 90)
 			(unlocked yes)
@@
 			)
 		)
-		(property "Value" "SMA002"
+		(property "Value" "6-1634010-0"
 			(at 2.5 1.5 90)
 			(unlocked yes)
@@
 			)
 		)
-		(property "Value" "SMA002"
+		(property "Value" "6-1634010-0"
 			(at 2.5 1.5 90)
 			(unlocked yes)
@@
 			)
 		)
-		(attr exclude_from_bom dnp)
+		(attr exclude_from_pos_files exclude_from_bom dnp)
 		(duplicate_pad_numbers_are_jumpers no)
 		(fp_poly
@@
 			)
 		)
-		(property "Value" "SMA002"
+		(property "Value" "6-1634010-0"
 			(at 2.5 1.5 90)
 			(unlocked yes)
@@
 			)
 		)
-		(property "MPN" "-"
+		(property "MPN" "DNP"
 			(at 0 0 90)
 			(unlocked yes)
@@
 			)
 		)
-		(property "old description" ""
+		(property "old description" "DNP: Do Not Populate (DNI)"
 			(at 0 0 90)
 			(unlocked yes)
@@
 			)
 		)
-		(attr exclude_from_bom dnp)
+		(attr exclude_from_pos_files exclude_from_bom)
 		(duplicate_pad_numbers_are_jumpers no)
 		(fp_line
@@
 			)
 		)
-		(property "MPN" ""
+		(property "MPN" "RC0402JR-070RL"
 			(at 0 0 0)
 			(unlocked yes)
@@
 			)
 		)
-		(property "OEPS PN" "OEPS020013"
+		(property "OEPS PN" "OEPS020001"
 			(at 0 0 0)
 			(unlocked yes)
@@
 			)
 		)
-		(property "old description" ""
+		(property "old description" "RESISTOR:   SMD 0402 0Ω 1A   [RC0402JR-070RL] [SMD]"
 			(at 0 0 0)
 			(unlocked yes)
@@
 			)
 		)
-		(property "MPN" ""
+		(property "MPN" "CC0402JRNPO9BN101"
 			(at 0 0 0)
 			(unlocked yes)
@@
 			)
 		)
-		(property "OEPS PN" ""
+		(property "OEPS PN" "OEPS010089"
 			(at 0 0 0)
 			(unlocked yes)
@@
 			)
 		)
-		(property "old description" ""
+		(property "old description" "CAPACITOR:   SMD CER 0402 100pF 50V ±5% C0G   [CC0402JRNPO9BN101] [SMD]"
 			(at 0 0 0)
 			(unlocked yes)
@@
 			)
 		)
-		(attr exclude_from_bom dnp)
+		(attr exclude_from_pos_files exclude_from_bom)
 		(duplicate_pad_numbers_are_jumpers no)
 		(pad "TP" smd roundrect
@@
 			)
 		)
-		(attr exclude_from_bom dnp)
+		(attr exclude_from_pos_files exclude_from_bom)
 		(duplicate_pad_numbers_are_jumpers no)
 		(pad "TP" smd roundrect
@@
 			)
 		)
-		(attr exclude_from_bom dnp)
+		(attr exclude_from_pos_files exclude_from_bom)
 		(duplicate_pad_numbers_are_jumpers no)
 		(pad "TP" smd roundrect
@@
 			)
 		)
-		(attr exclude_from_bom dnp)
+		(attr exclude_from_pos_files exclude_from_bom)
 		(duplicate_pad_numbers_are_jumpers no)
 		(pad "TP" smd roundrect
@@
 			)
 		)
-		(property "Value" "24ST"
+		(property "Value" "24AA64-I/ST"
 			(at 2.925 -3.25 0)
 			(unlocked yes)
@@
 			)
 		)
-		(attr exclude_from_bom dnp)
+		(attr exclude_from_pos_files exclude_from_bom)
 		(duplicate_pad_numbers_are_jumpers no)
 		(pad "TP" smd roundrect
@@
 			)
 		)
-		(property "Value" "LM4132AMF-2.5/NOPBCT-ND"
+		(property "Value" "LM4132AMF-2.5/NOPB"
 			(at -1.705 -3.0734 270)
 			(unlocked yes)
@@
 			)
 		)
-		(attr exclude_from_bom dnp)
+		(attr exclude_from_pos_files exclude_from_bom)
 		(duplicate_pad_numbers_are_jumpers no)
 		(pad "TP" smd roundrect
@@
 			)
 		)
-		(attr exclude_from_bom dnp)
+		(attr exclude_from_pos_files exclude_from_bom)
 		(duplicate_pad_numbers_are_jumpers no)
 		(pad "TP" smd roundrect
@@
 			)
 		)
-		(attr exclude_from_bom dnp)
+		(attr exclude_from_pos_files exclude_from_bom)
 		(duplicate_pad_numbers_are_jumpers no)
 		(pad "TP" smd roundrect
@@
 			)
 		)
-		(attr exclude_from_bom dnp)
+		(attr exclude_from_pos_files exclude_from_bom)
 		(duplicate_pad_numbers_are_jumpers no)
 		(pad "TP" smd roundrect
@@
 			)
 		)
-		(attr exclude_from_bom dnp)
+		(attr exclude_from_pos_files exclude_from_bom)
 		(duplicate_pad_numbers_are_jumpers no)
 		(pad "TP" smd roundrect
@@
 			)
 		)
-		(attr exclude_from_bom dnp)
+		(attr exclude_from_pos_files exclude_from_bom)
 		(duplicate_pad_numbers_are_jumpers no)
 		(pad "TP" smd roundrect
@@
 			)
 		)
-		(attr exclude_from_bom dnp)
+		(attr exclude_from_pos_files exclude_from_bom)
 		(duplicate_pad_numbers_are_jumpers no)
 		(pad "TP" smd roundrect
@@
 			)
 		)
-		(attr exclude_from_bom dnp)
+		(attr exclude_from_pos_files exclude_from_bom)
 		(duplicate_pad_numbers_are_jumpers no)
 		(pad "TP" smd roundrect
@@
 			)
 		)
-		(attr exclude_from_bom dnp)
+		(attr exclude_from_pos_files exclude_from_bom)
 		(duplicate_pad_numbers_are_jumpers no)
 		(pad "TP" smd roundrect
@@
 			)
 		)
-		(attr exclude_from_bom dnp)
+		(attr exclude_from_pos_files exclude_from_bom)
 		(duplicate_pad_numbers_are_jumpers no)
 		(pad "TP" smd roundrect
@@
 			)
 		)
-		(attr exclude_from_bom dnp)
+		(attr exclude_from_pos_files exclude_from_bom)
 		(duplicate_pad_numbers_are_jumpers no)
 		(pad "TP" smd roundrect
@@
 			)
 		)
-		(attr exclude_from_bom dnp)
+		(attr exclude_from_pos_files exclude_from_bom)
 		(duplicate_pad_numbers_are_jumpers no)
 		(pad "TP" smd roundrect
@@
 			)
 		)
-		(attr exclude_from_bom dnp)
+		(attr exclude_from_pos_files exclude_from_bom)
 		(duplicate_pad_numbers_are_jumpers no)
 		(pad "TP" smd roundrect
