File: pcb/fmc-host.kicad_sch (KiCad schematic)
At the start: 310 parts, among them J1 SMA002, J10 BM08B-SURS-TF, J2 SMA002, J3 SMA002, J4 SMA002, J5 SMA002, J6 FTSH-105-01-F-D-RA-K, J7 12226-8250-00FR, J8 FMC_SINGLE_WIDTH_MODULE, J9 ASP-134488-01, Q1 SI1012R, Q2 SI1012R, U1 SN74LVC2G34DCKR, U10 DS90UB934-Q1, U11 DS91M040, U12 AD5766BCPZ-RL7, U13 MCP47FEB02A0-E/ST, U14 LM4132AMF-2.5/NOPBCT-ND, U15 AD7616BSTZ, U16 AD5142BCPZ10, U17 LTM4622A, U18 D3V3XA4B10LP, U19 TPS7A49, U2 SN65LVDS9638DGN, U20 TPS7A49, U21 TPS7A30, U22 24ST, U23 LTM8049_BGA, U24 TPS62061DSGT, U25 D3V3XA4B10LP, U26 D3V3XA4B10LP, U3 FIN1032MTCX, U4 ADCMP600, U5 ADCMP600, U6 DG1412E, U7 DG1412E, U8 DG1412E, U9 DS90UB934-Q1, X2 OE-LOGO_7X5

Commit message: Updated OEPS PN.
Added OEPS PN to all components.
The cross-check between BOM and PNP files failed due to TP (test points) attributes.
Fixed TP attributes.
Added .history/ to .gitignore to remove KiCAD history files.
Parts:
- C115: MPN (none) -> CC0402JRNPO9BN101; OEPS PN (none) -> OEPS010089; old description (none) -> CAPACITOR: SMD CER 0402 100pF 50V ±5% C0G [CC0402JRNPO9BN10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
- D1, D2: value SESD0402X1UN-0020-090 -> SESD0402X1UN-0030-088
- D3, D4, D5: old description #N/A -> DIODE: RF DIODE PIN 150V 250MW [BAR66E6327HTSA1] [PG-SOT23]
- D6: value KDZ4.3B -> KDZVTR4.3B
- J1, J2, J3, J4, J5: value SMA002 -> 6-1634010-0
- L5, L6: value SRNxx-101M -> SRN6045TA-101M
- R34, R36: MPN - -> DNP; old description (none) -> DNP: Do Not Populate (DNI)
- R66: MPN (none) -> RC0402JR-070RL; OEPS PN (none) -> OEPS020001; old description (none) -> RESISTOR: SMD 0402 0Ω 1A [RC0402JR-070RL] [SMD]
- TP1, TP10, TP11, TP12, TP13, TP14, TP15, TP16, TP17, TP18, TP2, TP3, TP4, TP5, TP6, TP7, TP8, TP9, X2: now fitted
- U14: value LM4132AMF-2.5/NOPBCT-ND -> LM4132AMF-2.5/NOPB
- U16: value AD5142BCPZ10 -> AD5142BRUZ10
- U22: value 24ST -> 24AA64-I/ST
- U23: value LTM8049_BGA -> LTM8049IY#PBF
Changed lines of the file:
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@@
 			)
 		)
-		(property "old description" "#N/A"
+		(property "old description" "DIODE:   RF DIODE PIN 150V 250MW   [BAR66E6327HTSA1] [PG-SOT23]"
 			(at 106.68 754.38 0)
 			(hide yes)
@@
 		(in_bom no)
 		(on_board yes)
-		(in_pos_files yes)
-		(dnp yes)
+		(in_pos_files no)
+		(dnp no)
 		(property "Reference" "TP14"
 			(at 462.28 745.49 90)
@@
 		(in_bom no)
 		(on_board yes)
-		(in_pos_files yes)
+		(in_pos_files no)
 		(dnp yes)
 		(property "Reference" "J8"
@@
 		(in_bom no)
 		(on_board yes)
-		(in_pos_files yes)
-		(dnp yes)
+		(in_pos_files no)
+		(dnp no)
 		(property "Reference" "TP2"
 			(at 579.12 240.03 90)
@@
 		(in_bom no)
 		(on_board yes)
-		(in_pos_files yes)
-		(dnp yes)
+		(in_pos_files no)
+		(dnp no)
 		(property "Reference" "TP10"
 			(at 744.22 1281.43 90)
@@
 			)
 		)
-		(property "Value" "SRNxx-101M"
+		(property "Value" "SRN6045TA-101M"
 			(at 147.32 1080.262 90)
 			(show_name no)
@@
 		(in_bom no)
 		(on_board yes)
-		(in_pos_files yes)
-		(dnp yes)
+		(in_pos_files no)
+		(dnp no)
 		(property "Reference" "TP6"
 			(at 238.76 661.67 90)
@@
 		(in_bom no)
 		(on_board yes)
-		(in_pos_files yes)
-		(dnp yes)
+		(in_pos_files no)
+		(dnp no)
 		(property "Reference" "TP16"
 			(at 792.48 1294.13 90)
@@
 			)
 		)
-		(property "Value" "SMA002"
+		(property "Value" "6-1634010-0"
 			(at 68.58 581.66 0)
 			(show_name no)
@@
 		(in_bom no)
 		(on_board yes)
-		(in_pos_files yes)
-		(dnp yes)
+		(in_pos_files no)
+		(dnp no)
 		(property "Reference" "TP15"
 			(at 415.29 119.38 90)
@@
 		(in_bom no)
 		(on_board yes)
-		(in_pos_files yes)
-		(dnp yes)
+		(in_pos_files no)
+		(dnp no)
 		(property "Reference" "TP9"
 			(at 734.06 1281.43 90)
@@
 		(in_bom no)
 		(on_board yes)
-		(in_pos_files yes)
-		(dnp yes)
+		(in_pos_files no)
+		(dnp no)
 		(property "Reference" "TP1"
 			(at 574.04 240.03 90)
@@
 			)
 		)
-		(property "Value" "SMA002"
+		(property "Value" "6-1634010-0"
 			(at 60.96 1315.72 0)
 			(show_name no)
@@
 		(in_bom no)
 		(on_board yes)
-		(in_pos_files yes)
-		(dnp yes)
+		(in_pos_files no)
+		(dnp no)
 		(property "Reference" "TP4"
 			(at 584.2 240.03 90)
@@
 			)
 		)
-		(property "Value" "SRNxx-101M"
+		(property "Value" "SRN6045TA-101M"
 			(at 147.32 1313.942 90)
 			(show_name no)
@@
 			)
 		)
-		(property "Value" "SESD0402X1UN-0020-090"
+		(property "Value" "SESD0402X1UN-0030-088"
 			(at 102.87 1327.15 90)
 			(show_name no)
@@
 		(in_bom no)
 		(on_board yes)
-		(in_pos_files yes)
-		(dnp yes)
+		(in_pos_files no)
+		(dnp no)
 		(property "Reference" "TP5"
 			(at 304.8 613.41 90)
@@
 		(in_bom no)
 		(on_board yes)
-		(in_pos_files yes)
-		(dnp yes)
+		(in_pos_files no)
+		(dnp no)
 		(property "Reference" "TP18"
 			(at 764.54 1281.43 90)
@@
 			)
 		)
-		(property "old description" "#N/A"
+		(property "old description" "DIODE:   RF DIODE PIN 150V 250MW   [BAR66E6327HTSA1] [PG-SOT23]"
 			(at 116.84 665.48 0)
 			(hide yes)
@@
 			)
 		)
-		(property "old description" "#N/A"
+		(property "old description" "DIODE:   RF DIODE PIN 150V 250MW   [BAR66E6327HTSA1] [PG-SOT23]"
 			(at 116.84 576.58 0)
 			(hide yes)
@@
 		(in_bom no)
 		(on_board yes)
-		(in_pos_files yes)
-		(dnp yes)
+		(in_pos_files no)
+		(dnp no)
 		(property "Reference" "TP13"
 			(at 447.04 753.11 90)
@@
 			)
 		)
-		(property "Value" "LTM8049_BGA"
+		(property "Value" "LTM8049IY#PBF"
 			(at 822.96 138.43 0)
 			(show_name no)
@@
 		(in_bom no)
 		(on_board yes)
-		(in_pos_files yes)
-		(dnp yes)
+		(in_pos_files no)
+		(dnp no)
 		(property "Reference" "TP8"
 			(at 238.76 593.09 90)
@@
 			)
 		)
-		(property "Value" "SMA002"
+		(property "Value" "6-1634010-0"
 			(at 68.58 759.46 0)
 			(show_name no)
@@
 			)
 		)
-		(property "Value" "SMA002"
+		(property "Value" "6-1634010-0"
 			(at 68.58 670.56 0)
 			(show_name no)
@@
 		(in_bom no)
 		(on_board yes)
-		(in_pos_files yes)
-		(dnp yes)
+		(in_pos_files no)
+		(dnp no)
 		(property "Reference" "TP11"
 			(at 772.16 1294.13 90)
@@
 			)
 		)
-		(property "MPN" ""
+		(property "MPN" "CC0402JRNPO9BN101"
 			(at 579.12 416.56 0)
 			(hide yes)
@@
 			)
 		)
-		(property "OEPS PN" ""
+		(property "OEPS PN" "OEPS010089"
 			(at 579.12 416.56 0)
 			(hide yes)
@@
 			)
 		)
-		(property "old description" ""
+		(property "old description" "CAPACITOR:   SMD CER 0402 100pF 50V ±5% C0G   [CC0402JRNPO9BN101] [SMD]"
 			(at 579.12 416.56 0)
 			(hide yes)
@@
 			)
 		)
-		(property "MPN" "-"
+		(property "MPN" "DNP"
 			(at 304.8 1292.86 0)
 			(hide yes)
@@
 			)
 		)
-		(property "old description" ""
+		(property "old description" "DNP: Do Not Populate (DNI)"
 			(at 304.8 1292.86 0)
 			(hide yes)
@@
 			)
 		)
-		(property "Value" "24ST"
+		(property "Value" "24AA64-I/ST"
 			(at 723.9 1247.14 0)
 			(show_name no)
@@
 			)
 		)
-		(property "Value" "SMA002"
+		(property "Value" "6-1634010-0"
 			(at 60.96 1082.04 0)
 			(show_name no)
@@
 			)
 		)
-		(property "MPN" "-"
+		(property "MPN" "DNP"
 			(at 299.72 1059.18 0)
 			(hide yes)
@@
 			)
 		)
-		(property "old description" ""
+		(property "old description" "DNP: Do Not Populate (DNI)"
 			(at 299.72 1059.18 0)
 			(hide yes)
@@
 			)
 		)
-		(property "Value" "KDZ4.3B"
+		(property "Value" "KDZVTR4.3B"
 			(at 318.77 631.19 0)
 			(show_name no)
@@
 			)
 		)
-		(property "Value" "SESD0402X1UN-0020-090"
+		(property "Value" "SESD0402X1UN-0030-088"
 			(at 102.87 1093.47 90)
 			(show_name no)
@@
 			)
 		)
-		(property "Value" "AD5142BCPZ10"
+		(property "Value" "AD5142BRUZ10"
 			(at 520.7 831.85 0)
 			(show_name no)
@@
 		(in_bom no)
 		(on_board yes)
-		(in_pos_files yes)
-		(dnp yes)
+		(in_pos_files no)
+		(dnp no)
 		(property "Reference" "X2"
 			(at 106.68 1356.36 0)
@@
 		(in_bom no)
 		(on_board yes)
-		(in_pos_files yes)
-		(dnp yes)
+		(in_pos_files no)
+		(dnp no)
 		(property "Reference" "TP3"
 			(at 594.36 240.03 90)
@@
 		(in_bom no)
 		(on_board yes)
-		(in_pos_files yes)
-		(dnp yes)
+		(in_pos_files no)
+		(dnp no)
 		(property "Reference" "TP12"
 			(at 782.32 1294.13 90)
@@
 			)
 		)
-		(property "MPN" ""
+		(property "MPN" "RC0402JR-070RL"
 			(at 609.6 408.94 0)
 			(hide yes)
@@
 			)
 		)
-		(property "old description" ""
+		(property "old description" "RESISTOR:   SMD 0402 0Ω 1A   [RC0402JR-070RL] [SMD]"
+			(at 609.6 408.94 0)
+			(hide yes)
+			(show_name no)
+			(do_not_autoplace no)
+			(effects
+				(font
+					(size 1.27 1.27)
+				)
+			)
+		)
+		(property "OEPS PN" "OEPS020001"
 			(at 609.6 408.94 0)
 			(hide yes)
@@
 		(in_bom no)
 		(on_board yes)
-		(in_pos_files yes)
-		(dnp yes)
+		(in_pos_files no)
+		(dnp no)
 		(property "Reference" "TP7"
 			(at 238.76 572.77 90)
@@
 			)
 		)
-		(property "Value" "LM4132AMF-2.5/NOPBCT-ND"
+		(property "Value" "LM4132AMF-2.5/NOPB"
 			(at 406.4 328.93 0)
 			(show_name no)
@@
 		(in_bom no)
 		(on_board yes)
-		(in_pos_files yes)
-		(dnp yes)
+		(in_pos_files no)
+		(dnp no)
 		(property "Reference" "TP17"
 			(at 754.38 1281.43 90)

Commit message: Update component part numbers and specifications
Parts:
- J1, J2, J3, J4, J5: MPN 6-1634010-0 -> 262105; OEPS PN OEPS070003 -> OEPS070081; old description CONNECTOR: MMCX RCPT 50ohm 90º [6-1634010-0] [TH] -> CONNECTOR: MMCX RCPT 50ohm 90º [262105] [TH]
- L1, L2: MPN 1008PS-472KLB -> 1008PS-472KLC; old description INDUCTOR: FIXED INDUCTOR SMD 4.7uH 950mA 350mΩ [1008PS-472KLB] [-] -> INDUCTOR: FIXED INDUCTOR SMD 4.7uH 950mA 350mΩ [1008PS-472KLC] [-]
- Q1, Q2: MPN SI1012R-T1-GE3 -> SI1012CR-T1-GE3; OEPS PN OEPS060001 -> OEPS060024; old description TRANSISTOR: MOSFET N-CH 20V 500mA [SI1012R-T1-GE3] [SC-75A] -> TRANSISTOR: MOSFET N-CH 20V 630mA [SI1012CR-T1-GE3] [SC-75A]
Changed lines of the file:
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@@
 			)
 		)
-		(property "MPN" "SI1012R-T1-GE3"
+		(property "MPN" "SI1012CR-T1-GE3"
 			(at 154.94 617.22 0)
 			(hide yes)
@@
 			)
 		)
-		(property "OEPS PN" "OEPS060001"
+		(property "OEPS PN" "OEPS060024"
 			(at 154.94 617.22 0)
 			(hide yes)
@@
 			)
 		)
-		(property "old description" "TRANSISTOR:   MOSFET N-CH 20V 500mA   [SI1012R-T1-GE3] [SC-75A]"
+		(property "old description" "TRANSISTOR:   MOSFET N-CH 20V 630mA   [SI1012CR-T1-GE3] [SC-75A]"
 			(at 154.94 617.22 0)
 			(hide yes)
@@
 			)
 		)
-		(property "MPN" "1008PS-472KLB"
+		(property "MPN" "1008PS-472KLC"
 			(at 124.46 1076.96 90)
 			(hide yes)
@@
 			)
 		)
-		(property "old description" "INDUCTOR:   FIXED INDUCTOR SMD 4.7uH 950mA 350mΩ   [1008PS-472KLB] [-]"
+		(property "old description" "INDUCTOR:   FIXED INDUCTOR SMD 4.7uH 950mA 350mΩ   [1008PS-472KLC] [-]"
 			(at 124.46 1076.96 90)
 			(hide yes)
@@
 			)
 		)
-		(property "MPN" "6-1634010-0"
+		(property "MPN" "262105"
 			(at 71.12 576.58 0)
 			(hide yes)
@@
 			)
 		)
-		(property "OEPS PN" "OEPS070003"
+		(property "OEPS PN" "OEPS070081"
 			(at 71.12 576.58 0)
 			(hide yes)
@@
 			)
 		)
-		(property "old description" "CONNECTOR:   MMCX RCPT 50ohm 90º   [6-1634010-0] [TH]"
+		(property "old description" "CONNECTOR:   MMCX RCPT 50ohm 90º   [262105] [TH]"
 			(at 71.12 576.58 0)
 			(hide yes)
@@
 			)
 		)
-		(property "MPN" "6-1634010-0"
+		(property "MPN" "262105"
 			(at 63.5 1310.64 0)
 			(hide yes)
@@
 			)
 		)
-		(property "OEPS PN" "OEPS070003"
+		(property "OEPS PN" "OEPS070081"
 			(at 63.5 1310.64 0)
 			(hide yes)
@@
 			)
 		)
-		(property "old description" "CONNECTOR:   MMCX RCPT 50ohm 90º   [6-1634010-0] [TH]"
+		(property "old description" "CONNECTOR:   MMCX RCPT 50ohm 90º   [262105] [TH]"
 			(at 63.5 1310.64 0)
 			(hide yes)
@@
 			)
 		)
-		(property "MPN" "6-1634010-0"
+		(property "MPN" "262105"
 			(at 71.12 754.38 0)
 			(hide yes)
@@
 			)
 		)
-		(property "OEPS PN" "OEPS070003"
+		(property "OEPS PN" "OEPS070081"
 			(at 71.12 754.38 0)
 			(hide yes)
@@
 			)
 		)
-		(property "old description" "CONNECTOR:   MMCX RCPT 50ohm 90º   [6-1634010-0] [TH]"
+		(property "old description" "CONNECTOR:   MMCX RCPT 50ohm 90º   [262105] [TH]"
 			(at 71.12 754.38 0)
 			(hide yes)
@@
 			)
 		)
-		(property "MPN" "6-1634010-0"
+		(property "MPN" "262105"
 			(at 71.12 665.48 0)
 			(hide yes)
@@
 			)
 		)
-		(property "OEPS PN" "OEPS070003"
+		(property "OEPS PN" "OEPS070081"
 			(at 71.12 665.48 0)
 			(hide yes)
@@
 			)
 		)
-		(property "old description" "CONNECTOR:   MMCX RCPT 50ohm 90º   [6-1634010-0] [TH]"
+		(property "old description" "CONNECTOR:   MMCX RCPT 50ohm 90º   [262105] [TH]"
 			(at 71.12 665.48 0)
 			(hide yes)
@@
 			)
 		)
-		(property "MPN" "1008PS-472KLB"
+		(property "MPN" "1008PS-472KLC"
 			(at 124.46 1310.64 90)
 			(hide yes)
@@
 			)
 		)
-		(property "old description" "INDUCTOR:   FIXED INDUCTOR SMD 4.7uH 950mA 350mΩ   [1008PS-472KLB] [-]"
+		(property "old description" "INDUCTOR:   FIXED INDUCTOR SMD 4.7uH 950mA 350mΩ   [1008PS-472KLC] [-]"
 			(at 124.46 1310.64 90)
 			(hide yes)
@@
 			)
 		)
-		(property "MPN" "6-1634010-0"
+		(property "MPN" "262105"
 			(at 63.5 1076.96 0)
 			(hide yes)
@@
 			)
 		)
-		(property "OEPS PN" "OEPS070003"
+		(property "OEPS PN" "OEPS070081"
 			(at 63.5 1076.96 0)
 			(hide yes)
@@
 			)
 		)
-		(property "old description" "CONNECTOR:   MMCX RCPT 50ohm 90º   [6-1634010-0] [TH]"
+		(property "old description" "CONNECTOR:   MMCX RCPT 50ohm 90º   [262105] [TH]"
 			(at 63.5 1076.96 0)
 			(hide yes)
@@
 			)
 		)
-		(property "MPN" "SI1012R-T1-GE3"
+		(property "MPN" "SI1012CR-T1-GE3"
 			(at 154.94 706.12 0)
 			(hide yes)
@@
 			)
 		)
-		(property "OEPS PN" "OEPS060001"
+		(property "OEPS PN" "OEPS060024"
 			(at 154.94 706.12 0)
 			(hide yes)
@@
 			)
 		)
-		(property "old description" "TRANSISTOR:   MOSFET N-CH 20V 500mA   [SI1012R-T1-GE3] [SC-75A]"
+		(property "old description" "TRANSISTOR:   MOSFET N-CH 20V 630mA   [SI1012CR-T1-GE3] [SC-75A]"
 			(at 154.94 706.12 0)
 			(hide yes)

Commit message: Address EDADOCs EQs for rev. g
Connections:
- net GND: now also J6.05 (5), J6.06 (6)
Changed lines of the file:
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@@
 	(wire
 		(pts
+			(xy 76.2 792.48) (xy 80.01 792.48)
+		)
+		(stroke
+			(width 0)
+			(type default)
+		)
+	)
+	(wire
+		(pts
 			(xy 713.74 1236.98) (xy 713.74 1239.52)
 		)
@@
 	(wire
 		(pts
+			(xy 76.2 822.96) (xy 76.2 792.48)
+		)
+		(stroke
+			(width 0)
+			(type default)
+		)
+	)
+	(wire
+		(pts
 			(xy 426.72 680.72) (xy 635 680.72)
 		)
@@
 		)
 	)
+	(wire
+		(pts
+			(xy 80.01 792.48) (xy 80.01 795.02)
+		)
+		(stroke
+			(width 0)
+			(type default)
+		)
+	)
 	(polyline
 		(pts
@@
 		)
 	)
+	(wire
+		(pts
+			(xy 76.2 838.2) (xy 76.2 853.44)
+		)
+		(stroke
+			(width 0)
+			(type default)
+		)
+	)
 	(polyline
 		(pts
@@
 	)
 	(symbol
+		(lib_id "fmc-host-eagle-import:GND")
+		(at 80.01 797.56 0)
+		(unit 1)
+		(body_style 1)
+		(exclude_from_sim no)
+		(in_bom yes)
+		(on_board yes)
+		(in_pos_files yes)
+		(dnp no)
+		(property "Reference" "#SUPPLY0212"
+			(at 80.01 797.56 0)
+			(hide yes)
+			(show_name no)
+			(do_not_autoplace no)
+			(effects
+				(font
+					(size 1.27 1.27)
+				)
+			)
+		)
+		(property "Value" "GND"
+			(at 75.565 802.259 0)
+			(show_name no)
+			(do_not_autoplace no)
+			(effects
+				(font
+					(size 1.778 1.5113)
+				)
+				(justify left bottom)
+			)
+		)
+		(property "Footprint" ""
+			(at 80.01 797.56 0)
+			(hide yes)
+			(show_name no)
+			(do_not_autoplace no)
+			(effects
+				(font
+					(size 1.27 1.27)
+				)
+			)
+		)
+		(property "Datasheet" ""
+			(at 80.01 797.56 0)
+			(hide yes)
+			(show_name no)
+			(do_not_autoplace no)
+			(effects
+				(font
+					(size 1.27 1.27)
+				)
+			)
+		)
+		(property "Description" ""
+			(at 80.01 797.56 0)
+			(hide yes)
+			(show_name no)
+			(do_not_autoplace no)
+			(effects
+				(font
+					(size 1.27 1.27)
+				)
+			)
+		)
+		(pin "1"
+		)
+		(instances
+			(project "fmc-host"
+				(path "/3a190272-84f9-4241-a964-a08ef93e1ba1"
+					(reference "#SUPPLY0212")
+					(unit 1)
+				)
+			)
+		)
+	)
+	(symbol
 		(lib_id "fmc-host-eagle-import:DIODE2_SOT23")
 		(at 116.84 665.48 0)
@@
 					(unit 1)
 				)
+			)
+		)
+	)
+	(symbol
+		(lib_id "fmc-host-eagle-import:GND")
+		(at 76.2 855.98 0)
+		(unit 1)
+		(body_style 1)
+		(exclude_from_sim no)
+		(in_bom yes)
+		(on_board yes)
+		(in_pos_files yes)
+		(dnp no)
+		(property "Reference" "#SUPPLY0113"
+			(at 76.2 855.98 0)
+			(hide yes)
+			(show_name no)
+			(do_not_autoplace no)
+			(effects
+				(font
+					(size 1.27 1.27)
+				)
+			)
+		)
+		(property "Value" "GND"
+			(at 71.755 860.679 0)
+			(show_name no)
+			(do_not_autoplace no)
+			(effects
+				(font
+					(size 1.778 1.5113)
+				)
+				(justify left bottom)
+			)
+		)
+		(property "Footprint" ""
+			(at 76.2 855.98 0)
+			(hide yes)
+			(show_name no)
+			(do_not_autoplace no)
+			(effects
+				(font
+					(size 1.27 1.27)
+				)
+			)
+		)
+		(property "Datasheet" ""
+			(at 76.2 855.98 0)
+			(hide yes)
+			(show_name no)
+			(do_not_autoplace no)
+			(effects
+				(font
+					(size 1.27 1.27)
+				)
+			)
+		)
+		(property "Description" ""
+			(at 76.2 855.98 0)
+			(hide yes)
+			(show_name no)
+			(do_not_autoplace no)
+			(effects
+				(font
+					(size 1.27 1.27)
+				)
+			)
+		)
+		(pin "1"
+		)
+		(instances
+			(project "fmc-host"
+				(path "/3a190272-84f9-4241-a964-a08ef93e1ba1"
+					(reference "#SUPPLY0113")
+					(unit 1)
+				)
