File: pcb/fmc-host.kicad_sch (KiCad schematic)
At the start: 310 parts, among them J1 6-1634010-0, J10 BM08B-SURS-TF, J2 6-1634010-0, J3 6-1634010-0, J4 6-1634010-0, J5 6-1634010-0, J6 FTSH-105-01-F-D-RA-K, J7 12226-8250-00FR, J8 FMC_SINGLE_WIDTH_MODULE, J9 ASP-134488-01, Q1 SI1012R, Q2 SI1012R, U1 SN74LVC2G34DCKR, U10 DS90UB934-Q1, U11 DS91M040, U12 AD5766BCPZ-RL7, U13 MCP47FEB02A0-E/ST, U14 LM4132AMF-2.5/NOPB, U15 AD7616BSTZ, U16 AD5142BRUZ10, U17 LTM4622A, U18 D3V3XA4B10LP, U19 TPS7A49, U2 SN65LVDS9638DGN, U20 TPS7A49, U21 TPS7A30, U22 24AA64-I/ST, U23 LTM8049IY#PBF, U24 TPS62061DSGT, U25 D3V3XA4B10LP, U26 D3V3XA4B10LP, U3 FIN1032MTCX, U4 ADCMP600, U5 ADCMP600, U6 DG1412E, U7 DG1412E, U8 DG1412E, U9 DS90UB934-Q1, X2 OE-LOGO_7X5

Commit message: Add optional active discharge circuit
- This circuit actively discharges Vlink when the power supply is
  disabled.
- It sinks up to ~440 mA through a 4.7ohm, 1W resistor
- Will discharge worst case headstage in 20 millseconds or so
Parts:
- added C141, C142: 0.1uF, Capacitor_SMD:C_0402_1005Metric, symbol Device:C
- added Q3, Q4: SI1012R, Package_TO_SOT_SMD:SOT-523, symbol Transistor_FET:Q_NMOS_GSD
- added R289, R290: 4.7,1W, Resistor_SMD:R_1206_3216Metric, symbol Device:R_US
- added R83, R84: 165k, Resistor_SMD:R_0402_1005Metric, symbol fmc-host-eagle-import:R_0402
- added U27: TLV9062IDSGR, Package_SON:WSON-8-1EP_2x2mm_P0.5mm_EP0.9x1.6mm, symbol Amplifier_Operational:TLV9062xDSG
- added U28: SN74LVC2G14DBV, Package_TO_SOT_SMD:SOT-23-6, symbol 74xGxx:SN74LVC2G14DBV
- Q1, Q2: symbol fmc-host-eagle-import:N-MOSFET_SC75-GSD -> Transistor_FET:Q_NMOS_GSD
Connections:
- net +3V3: now also C141.1, C142.1, U27.8 (V+), U28.5 (V_{CC})
- net GND: now also C141.2, C142.2, R289.2, R290.2, R83.1, R84.1, U27.4 (V-), U27.9 (PAD), U28.2 (GND)
- net LINK_A_PWR_EN: now also U28.1 (1A)
- net LINK_B_PWR_EN: now also U28.3 (2A)
- net LVDS_DIN0_N: now also U18.10 (NC)
- net LVDS_DIN0_P: now also U18.9 (NC)
- net LVDS_DIN1_N: now also U18.6 (NC)
- net LVDS_DIN1_P: now also U18.7 (NC)
- net LVDS_DOUT0_N: now also U26.7 (NC)
- net LVDS_DOUT0_P: now also U26.6 (NC)
- net LVDS_DOUT1_N: now also U26.10 (NC)
- net LVDS_DOUT1_P: now also U26.9 (NC)
- net VLINK_A: now also Q3.3 (D)
- net VLINK_B: now also Q4.3 (D)
- new net: Q4.2 (S), R290.1, U27.6 (-)
- new net: U27.5 (+), U28.4 (2Y)
- new net: U27.3 (+), U28.6 (1Y)
- new net: Q4.1 (G), R84.2, U27.7
- new net: Q3.2 (S), R289.1, U27.2 (-)
- new net: Q3.1 (G), R83.2, U27.1
Other:
- moved on the sheet: U26

Commit message: Update component's annotation
Ready to generate BOM and PnP files.
Parts:
- C141, C142: MPN C1005X7R1E104K050BB -> GRM155R71E104KE14D; OEPS PN (none) -> OEPS010004; old description (none) -> CAPACITOR: SMD CER 0402 100nF 25V ±10% X7R [GRM155R71E104KE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
- R289, R290: OEPS PN (none) -> OEPS020260; old description (none) -> RESISTOR: SMD 1206 4.7Ω ±5% 1W [SG73P2BTTD4R7J] [SMD]
- U27: OEPS PN (none) -> OEPS080246; old description (none) -> IC: OPAMP 2 CIRCUIT [TLV9062IDSGR] [8-WSON]
- U28: MPN SN74LVC2G14DBV -> SN74LVC2G14DBVR; OEPS PN (none) -> OEPS080247; old description (none) -> IC: BUFFER INVERT 2CH SCHMITT-TRIGGER [SN74LVC2G14DBVR] [SO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
Changed lines of the file:
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@@
 			)
 		)
+		(property "OEPS PN" "OEPS020260"
+			(at 549.91 734.06 90)
+			(hide yes)
+			(show_name no)
+			(do_not_autoplace no)
+			(effects
+				(font
+					(size 1.27 1.27)
+				)
+			)
+		)
+		(property "old description" "RESISTOR:   SMD 1206 4.7Ω ±5% 1W   [SG73P2BTTD4R7J] [SMD]"
+			(at 549.91 734.06 90)
+			(hide yes)
+			(show_name no)
+			(do_not_autoplace no)
+			(effects
+				(font
+					(size 1.27 1.27)
+				)
+			)
+		)
 		(pin "1"
 		)
@@
 			)
 		)
-		(property "MPN" "SN74LVC2G14DBV"
+		(property "MPN" "SN74LVC2G14DBVR"
+			(at 605.79 713.74 0)
+			(hide yes)
+			(show_name no)
+			(do_not_autoplace no)
+			(effects
+				(font
+					(size 1.27 1.27)
+				)
+			)
+		)
+		(property "OEPS PN" "OEPS080247"
+			(at 605.79 713.74 0)
+			(hide yes)
+			(show_name no)
+			(do_not_autoplace no)
+			(effects
+				(font
+					(size 1.27 1.27)
+				)
+			)
+		)
+		(property "old description" "IC:   BUFFER INVERT 2CH SCHMITT-TRIGGER   [SN74LVC2G14DBVR] [SOT-23-6]"
 			(at 605.79 713.74 0)
 			(hide yes)
@@
 			)
 		)
+		(property "OEPS PN" "OEPS080246"
+			(at 571.5 721.36 0)
+			(hide yes)
+			(show_name no)
+			(do_not_autoplace no)
+			(effects
+				(font
+					(size 1.27 1.27)
+				)
+			)
+		)
+		(property "old description" "IC:   OPAMP 2 CIRCUIT   [TLV9062IDSGR] [8-WSON]"
+			(at 571.5 721.36 0)
+			(hide yes)
+			(show_name no)
+			(do_not_autoplace no)
+			(effects
+				(font
+					(size 1.27 1.27)
+				)
+			)
+		)
 		(pin "1"
 		)
@@
 			)
 		)
-		(property "MPN" "C1005X7R1E104K050BB"
+		(property "MPN" "GRM155R71E104KE14D"
 			(at 613.41 698.5 0)
 			(hide yes)
@@
 			)
 		)
+		(property "OEPS PN" "OEPS010004"
+			(at 613.41 698.5 90)
+			(hide yes)
+			(show_name no)
+			(do_not_autoplace no)
+			(effects
+				(font
+					(size 1.27 1.27)
+				)
+			)
+		)
+		(property "old description" "CAPACITOR:   SMD CER 0402 100nF 25V ±10% X7R   [GRM155R71E104KE14D] [SMD]"
+			(at 613.41 698.5 90)
+			(hide yes)
+			(show_name no)
+			(do_not_autoplace no)
+			(effects
+				(font
+					(size 1.27 1.27)
+				)
+			)
+		)
 		(pin "1"
 		)
@@
 			)
 		)
+		(property "OEPS PN" "OEPS020260"
+			(at 474.98 726.44 90)
+			(hide yes)
+			(show_name no)
+			(do_not_autoplace no)
+			(effects
+				(font
+					(size 1.27 1.27)
+				)
+			)
+		)
+		(property "old description" "RESISTOR:   SMD 1206 4.7Ω ±5% 1W   [SG73P2BTTD4R7J] [SMD]"
+			(at 474.98 726.44 90)
+			(hide yes)
+			(show_name no)
+			(do_not_autoplace no)
+			(effects
+				(font
+					(size 1.27 1.27)
+				)
+			)
+		)
 		(pin "1"
 		)
@@
 			)
 		)
+		(property "OEPS PN" "OEPS080246"
+			(at 511.81 713.74 0)
+			(hide yes)
+			(show_name no)
+			(do_not_autoplace no)
+			(effects
+				(font
+					(size 1.27 1.27)
+				)
+			)
+		)
+		(property "old description" "IC:   OPAMP 2 CIRCUIT   [TLV9062IDSGR] [8-WSON]"
+			(at 511.81 713.74 0)
+			(hide yes)
+			(show_name no)
+			(do_not_autoplace no)
+			(effects
+				(font
+					(size 1.27 1.27)
+				)
+			)
+		)
 		(pin "1"
 		)
@@
 			)
 		)
-		(property "MPN" "C1005X7R1E104K050BB"
+		(property "MPN" "GRM155R71E104KE14D"
 			(at 509.27 703.58 0)
 			(hide yes)
@@
 			)
 		)
+		(property "OEPS PN" "OEPS010004"
+			(at 509.27 703.58 0)
+			(hide yes)
+			(show_name no)
+			(do_not_autoplace no)
+			(effects
+				(font
+					(size 1.27 1.27)
+				)
+			)
+		)
+		(property "old description" "CAPACITOR:   SMD CER 0402 100nF 25V ±10% X7R   [GRM155R71E104KE14D] [SMD]"
+			(at 509.27 703.58 0)
+			(hide yes)
+			(show_name no)
+			(do_not_autoplace no)
+			(effects
+				(font
+					(size 1.27 1.27)
+				)
+			)
+		)
 		(pin "1"
 		)
@@
 			(at 511.81 713.74 0)
 			(hide yes)
+			(show_name no)
+			(do_not_autoplace no)
+			(effects
+				(font
+					(size 1.27 1.27)
+				)
+			)
+		)
+		(property "OEPS PN" "OEPS080246"
+			(at 511.81 713.74 0)
+			(hide yes)
+			(show_name no)
+			(do_not_autoplace no)
+			(effects
+				(font
+					(size 1.27 1.27)
+				)
+			)
+		)
+		(property "old description" "IC:   OPAMP 2 CIRCUIT   [TLV9062IDSGR] [8-WSON]"
+			(at 511.81 713.74 0)
+			(hide yes)

Commit message: Make footprints consistent across parts
- Given part numbers now use the same, eagle-based footprints when that
  option is available
Parts:
- C141, C142: footprint Capacitor_SMD:C_0402_1005Metric -> fmc-host:0402
- Q3, Q4: footprint Package_TO_SOT_SMD:SOT-523 -> fmc-host:SC75
- R83, R84: footprint Resistor_SMD:R_0402_1005Metric -> fmc-host:0402
Changed lines of the file:
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@@
 			)
 		)
-		(property "Footprint" "Capacitor_SMD:C_0402_1005Metric"
+		(property "Footprint" "fmc-host:0402"
 			(at 617.22 699.4652 0)
 			(hide yes)
@@
 			)
 		)
-		(property "Footprint" "Resistor_SMD:R_0402_1005Metric"
+		(property "Footprint" "fmc-host:0402"
 			(at 563.88 736.6 0)
 			(hide yes)
@@
 			)
 		)
-		(property "Footprint" "Package_TO_SOT_SMD:SOT-523"
+		(property "Footprint" "fmc-host:SC75"
 			(at 547.37 718.82 0)
 			(hide yes)
@@
 			)
 		)
-		(property "Footprint" "Resistor_SMD:R_0402_1005Metric"
+		(property "Footprint" "fmc-host:0402"
 			(at 501.65 722.63 0)
 			(hide yes)
@@
 			)
 		)
-		(property "Footprint" "Package_TO_SOT_SMD:SOT-523"
+		(property "Footprint" "fmc-host:SC75"
 			(at 472.44 711.2 0)
 			(hide yes)
@@
 			)
 		)
-		(property "Footprint" "Capacitor_SMD:C_0402_1005Metric"
+		(property "Footprint" "fmc-host:0402"
 			(at 510.2352 707.39 0)
 			(hide yes)

Commit message: Add final production files. Ready for production.
- Deleted old OEPSPN Field (not being used).
- Updated BOM generation according to standard.
- Added revG to schematic and project properties.
- Added/fixed OEPS Description.
- Updated PCB with OEPS Description.
- Regenerated assembly PnP files and merge into one single file.
- Regenerated BOM and removed duplicated lines.
- Deleted Edadoc EQ that is now solved.

New parts added:
C141, C142 - OEPS010004 GRM155R71E104KE14D
U27, U28 - OEPS080246 TLV9062IDSGR
Q3, Q4 - OEPS060024 SI1012CR-T1-GE3
R83, R84 - OEPS020020 ERJ-2RKF1653X
R289, R290 - OEPS020260 SG73P2BTTD4R7J
Parts:
- C1, C106, C118, C139, C140, C2, C26, C27, C34, C35, C36, C37, C5, C6, C70, C71, C72, C73, C79, C80, C81, C91, C92: OEPS Description (none) -> CAPACITOR: SMD CER 1206 10uF 25V ±10% X7R [GRM31CR71E106KA1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
- C10, C100, C104, C107, C110, C111, C112, C114, C13, C132, C134, C135, C137, C138, C14, C15, C16, C17, C18, C19, C22, C23, C3, C30, C31, C32, C33, C4, C41, C43, C44, C45, C46, C47, C48, C49, C52, C53, C54, C55, C56, C60, C61, C63, C65, C67, C68, C7, C78, C8, C83, C84, C85, C86, C87, C89, C9, C90, C93, C99: OEPS Description (none) -> CAPACITOR: SMD CER 0402 100nF 25V ±10% X7R [GRM155R71E104KE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; TempCo (none) -> X7R; Voltage (none) -> 25V
- C101, C103, C105, C108, C109, C113, C116, C117, C119, C120, C121, C125, C126, C127, C59, C62, C69, C77, C95, C96: OEPS Description (none) -> CAPACITOR: SMD CER 0805 10uF 25V ±10% X5R [GRM21BR61E106KA7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
- C102, C130, C131, C94, C97, C98: OEPS Description (none) -> CAPACITOR: SMD CER 1210 47uF 25V ±20% X5R [TMK325ABJ476MM-T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
- C11, C12, C122, C123, C124, C20, C21, C24, C25, C50, C51, C57, C58, C82: OEPS Description (none) -> CAPACITOR: SMD CER 0402 10nF 25V ±10% X7R [GCM155R71E103KA3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
- C115: OEPS Description (none) -> CAPACITOR: SMD CER 0402 100pF 50V ±5% C0G [CC0402JRNPO9BN10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
- C128, C129: OEPS Description (none) -> CAPACITOR: SMD CER 1210 100nF 500V ±10% X7R [C1210C104KCRAC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
- C133, C136: OEPS Description (none) -> CAPACITOR POL: SMD TANT B0 1411 33uF 20V ±20% 50Ohm [TL8B03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
- C141, C142: LCSC C105883 -> (none); OEPS Description (none) -> CAPACITOR: SMD CER 0402 100nF 25V ±10% X7R [GRM155R71E104KE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; OEPSPN OEPS010050 -> (none)
- C28, C29: OEPS Description (none) -> CAPACITOR: SMD CER 0402 4.7nF 25V ±10% X7R [CC0402KRX7R8BB4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
- C38, C39: OEPS Description (none) -> CAPACITOR: SMD CER 0402 47nF 25V ±10% X7R [GRM155R71E473KA8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
- C40, C42, C64, C66, C74, C75, C76, C88: OEPS Description (none) -> CAPACITOR: SMD CER 0805 1uF 25V ±10% X7R [GCM21BR71E105KA56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
- D1, D2: OEPS Description (none) -> DIODE: TVS DIODE 7VWM 13VC [SESD0402X1UN-0030-088] [0402/2D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
- D3, D4, D5: OEPS Description (none) -> DIODE: RF DIODE PIN 150V 250MW [BAR66E6327HTSA1] [PG-SOT23]
- D6: OEPS Description (none) -> DIODE: DIODE ZENER 4.55V 1W [KDZVTR4.3B] [PMDU]
- F1, F2, F3: OEPS Description (none) -> OTHER: PTC RESET FUSE 60V 140MA 1812 [MINISMDC014F-2] [Othe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
- J1, J2, J3, J4, J5: OEPS Description (none) -> CONNECTOR: MMCX RCPT 50ohm 90º [262105] [TH]
- J10: OEPS Description (none) -> CONNECTOR: HEADER 0.8MM 8POS [BM08B-SURS-TF] [SMD]
- J6: OEPS Description (none) -> CONNECTOR: HEADER 1.27MM R/A 10POS [FTSH-105-01-F-D-RA-K] [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
- J7: OEPS Description (none) -> CONNECTOR: SDR RCPT 90º 26POS [12226-8250-00FR] [SMD]
- J9: OEPS Description (none) -> CONNECTOR: ARRAY PLUG 400POS GOLD [ASP-134488-01] [SMD]
- L1, L2: OEPS Description (none) -> INDUCTOR: FIXED INDUCTOR SMD 4.7uH 950mA 350mΩ [1008PS-472K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
- L10, L11, L12, L3, L4, L9: OEPS Description (none) -> INDUCTOR: FERRITE BEAD SMD 0603 600Ω 1.3A 150mΩ (OEPS J30 0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
- L13: OEPS Description (none) -> INDUCTOR: FIXED INDUCTOR SMD 6.8uH 1.2A 276mΩ [1277AS-H-6R8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
- L14, L15, L16, L17, L18, L19: OEPS Description (none) -> INDUCTOR: FERRITE BEAD SMD 0402 600Ω 900mA 230mΩ [BLM15PX60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
- L5, L6: OEPS Description (none) -> INDUCTOR: FIXED INDUCTOR SMD 100uH 920mA 456mΩ [SRN6045TA-1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
- L7, L8: OEPS Description (none) -> INDUCTOR: FERRITE BEAD SMD 0805 1kΩ 1.5A 150mΩ [MPZ2012S102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
- Q1, Q2, Q3, Q4: OEPS Description (none) -> TRANSISTOR: MOSFET N-CH 20V 630mA [SI1012CR-T1-GE3] [SC-75A]
- R1, R2, R38, R39: OEPS Description (none) -> RESISTOR: SMD 0402 3kΩ ±1% 0.100W [ERJ-2RKF3001X] [SMD]
- R10, R3, R4, R57, R58, R9: OEPS Description (none) -> RESISTOR: SMD 0402 2kΩ ±1% 0.100W [ERJ-2RKF2001X] [SMD]
- R11, R12, R5, R6, R7, R8: OEPS Description (none) -> RESISTOR: SMD 0603 150Ω ±1% 0.250W [CRGP0603F150R] [SMD]
- R13, R14, R49, R50, R51, R52, R76, R83, R84: OEPS Description (none) -> RESISTOR: SMD 0402 165kΩ ±1% 0.100W [ERJ-2RKF1653X] [SMD]
- R15, R16, R35, R37, R59, R63, R64, R65, R67, R68, R78, R79, R82: OEPS Description (none) -> RESISTOR: SMD 0402 10kΩ ±1% 0.100W [ERJ-2RKF1002X] [SMD]
- R17, R18, R41, R42, R44, R45, R46, R47: OEPS Description (none) -> RESISTOR: SMD 0402 1kΩ ±1% 0.100W [ERJ-2RKF1001X] [SMD]
- R19, R21: OEPS Description (none) -> RESISTOR: SMD 0402 5.6kΩ ±1% 0.100W [ERJ-2RKF5601X] [SMD]
- R20, R22: OEPS Description (none) -> RESISTOR: SMD 0402 21kΩ ±1% 0.100W [ERJ-2RKF2102X] [SMD]
- R23, R24, R28, R29: OEPS Description (none) -> RESISTOR: SMD 0402 49.9Ω ±0.5% 0.063W [RR0510R-49R9-D] [SMD]
- R25, R26, R27: OEPS Description (none) -> RESISTOR: SMD 0402 100Ω ±1% 0.100W [ERJ-2RKF1000X] [SMD]
- R289, R290: OEPS Description (none) -> RESISTOR: SMD 1206 4.7Ω ±5% 1W [SG73P2BTTD4R7J] [SMD]
- R30, R31, R32, R33, R40, R43, R71, R73, R75: OEPS Description (none) -> RESISTOR: SMD 0402 4.7kΩ ±1% 0.100W [ERJ-2RKF4701X] [SMD]
- R34, R36: OEPS Description (none) -> DNP: Do Not Populate (DNI)
- R48, R66: OEPS Description (none) -> RESISTOR: SMD 0402 0Ω 1A [RC0402JR-070RL] [SMD]
- R53, R54, R55, R56: OEPS Description (none) -> IC: RES ARRAY 8 RES 2.2K OHM 1506 [EXB-2HV222JV] [SMD]
- R60, R61: OEPS Description (none) -> RESISTOR: SMD 0402 3.48kΩ ±1% 0.100W [ERJ-2RKF3481X] [SMD]
- R62: OEPS Description (none) -> RESISTOR: SMD 0402 649kΩ ±1% 0.100W [ERJ-2RKF6493X] [SMD]
- R69: OEPS Description (none) -> RESISTOR: SMD 0402 2.2kΩ ±1% 0.100W [ERJ-2RKF2201X] [SMD]
- R70: OEPS Description (none) -> RESISTOR: SMD 0402 15kΩ ±1% 0.100W [ERJ-2RKF1502X] [SMD]
- R72, R74: OEPS Description (none) -> RESISTOR: SMD 0402 47kΩ ±1% 0.100W [ERJ-2RKF4702X] [SMD]
- R77: OEPS Description (none) -> RESISTOR: SMD 0402 178kΩ ±1% 0.100W [ERJ-2RKF1783X] [SMD]
- R80, R81: OEPS Description (none) -> RESISTOR: SMD 0402 73.2kΩ ±1% 0.100W [ERJ-2RKF7322X] [SMD]
- S1, S2: OEPS Description (none) -> OTHER: SWITCH SLIDE DIP SPST 0.1A 6V 1 POS [CHS-01TA] [Othe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
- S3: OEPS Description (none) -> OTHER: SWITCH SLIDE DIP SPST 0.1A 6V 2 POS [CHS-02TB] [Othe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
- U1: OEPS Description (none) -> IC: BUFFER NON-INVERT 2CH [SN74LVC2G34DCKR] [SC-70-6]
- U10, U9: OEPS Description (none) -> IC: DESERIALIZER FPD-Link III [DS90UB934TRGZRQ1] [48-VQFN (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
- U11: OEPS Description (none) -> IC: TRANSCEIVER Half LVDS [DS91M040TSQ/NOPB] [32-WQFN (5x5)]
- U12: OEPS Description (none) -> IC: DAC 16BIT 16CH [AD5766BCPZ-RL7] [40-LFCSP-WQ (6x6)]
- U13: OEPS Description (none) -> IC: DAC 8BIT 2CH [MCP47FEB02A0-E/ST] [8-TSSOP]
- U14: OEPS Description (none) -> IC: VREF 2.5V 0.05% [LM4132AMF-2.5/NOPB] [SOT-23-5]
- U15: OEPS Description (none) -> IC: ADC 16BIT 16 channels [AD7616BSTZ] [80-LQFP]
- U16: OEPS Description (none) -> IC: DGT POT 10KOHM 256TAP 16TSSOP [AD5142BRUZ10] [16-TSSOP]
- U17: OEPS Description (none) -> IC: DC-DC CONVERTER 2outputs1.5-12V 1.5-12V [LTM4622AIY#PBF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
- U18, U25, U26: OEPS Description (none) -> IC: TVS DIODE ARRAY [D3V3XA4B10LP-7] [10-UFDFN]
- U19, U20: OEPS Description (none) -> IC: LDO ADJ 150mA [TPS7A4901DRBR] [8-SON (3x3)]
- U2: OEPS Description (none) -> IC: LVDS 2channel driver [SN65LVDS9638DGN] [8-MSOP-PowerPad]
- U21: OEPS Description (none) -> IC: LDO NEGATIVE ADJ 200mA [TPS7A3001DRBT] [8-SON (3x3)]
- U22: OEPS Description (none) -> IC: EEPROM 64KBIT I2C [24AA64-I/ST] [8-TSSOP]
- U23: OEPS Description (none) -> IC: DC DC CONVERTER ADJ 2outputs 2x1A [LTM8049IY#PBF] [77-B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
- U24: OEPS Description (none) -> IC: FIXED REG BUCK 1.8V 1.6A [TPS62061DSGT] [8-WSON (2x2)]
- U27: OEPS Description (none) -> IC: OPAMP 2 CIRCUIT [TLV9062IDSGR] [8-WSON]
- U28: OEPS Description (none) -> IC: BUFFER INVERT 2CH SCHMITT-TRIGGER [SN74LVC2G14DBVR] [SO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
- U3: OEPS Description (none) -> IC: LVDS 4channel receiver [FIN1032MTCX] [16-TSSOP]
- U4, U5: OEPS Description (none) -> IC: COMPARATOR 1 GP [ADCMP600BRJZ-R2] [SOT23-5]
- U6, U7, U8: OEPS Description (none) -> IC: SWITCH SPST-NOX4 1.5OHM [DG1412EEN-T1-GE4] [16-QFN (4x4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
